File: hardware/kicad/8088-mainboard/8088-mainboard.kicad_pcb (KiCad board)
At the start: 2 copper layers, 163 x 137 mm, 66 parts, among them J1 POWER 5v, J2 Exp0, J3 Exp1, SW1 Reset, U1 8088, U10 74LS273, U11 74LS00, U12 74LS138, U13 HM62256BLP, U14 74LS373, U15 74LS00, U2 8284, U3 74LS373, U4 74LS373, U5 74LS245, U6 8288, U7 74LS138, U8 28C256, U9 HM62256BLP, Y1 14.31818 MHz

Commit message: Update 8086-mainboard scheme
Parts:
- removed C5: 100nF, Capacitor_THT:C_Disc_D5.0mm_W2.5mm_P5.00mm
- removed U4: 74LS373, Package_DIP:DIP-20_W7.62mm
- U1: value 8088 -> 8088_Max_Mode
- moved C4 103.0 mm to (51.8, 35.5)
- moved R1 88.2 mm to (59.7, 30.7)
- moved C18 22.5 mm to (103.9, 93.3)
- moved C7 22.5 mm to (103.9, 70.8)
- moved U15 22.5 mm to (104.4, 128.3)
- moved C6 22.5 mm to (103.9, 48.2)
- moved U3 22.5 mm to (104.4, 60.8)
- moved C19 22.5 mm to (103.9, 115.8)
- moved U5 22.5 mm to (104.4, 83.3)
- moved U14 22.5 mm to (104.4, 105.8)
- moved J_DEBUG1 9.03 mm to (123.6, 25.6)
- moved C8 4.99 mm to (40.5, 52.7), turned to 90 degrees
Connections:
- net /A0 renamed /CPU/A0
- net /A1 renamed /CPU/A1
- net /A16 renamed /CPU/A16
- net /A17 renamed /CPU/A17
- net /A18 renamed /CPU/A18
- net /A19 renamed /CPU/A19
- net /A2 renamed /CPU/A2
- net /A3 renamed /CPU/A3
- net /A4 renamed /CPU/A4
- net /A5 renamed /CPU/A5
- net /A6 renamed /CPU/A6
- net /A7 renamed /CPU/A7
- net /D0 renamed /CPU/D0
- net /D1 renamed /CPU/D1
- net /D2 renamed /CPU/D2
- net /D3 renamed /CPU/D3
- net /D4 renamed /CPU/D4
- net /D5 renamed /CPU/D5
- net /D6 renamed /CPU/D6
- net /D7 renamed /CPU/D7
- J2 pad 19: /A9 -> /CPU/A9
- J2 pad 20: /A8 -> /CPU/A8
- J2 pad 21: /A11 -> /CPU/A11
- J2 pad 22: /A10 -> /CPU/A10
- J2 pad 23: /A13 -> /CPU/A13
- J2 pad 24: /A12 -> /CPU/A12
- J2 pad 25: /A15 -> /CPU/A15
- J2 pad 26: /A14 -> /CPU/A14
- J3 pad 19: /A9 -> /CPU/A9
- J3 pad 20: /A8 -> /CPU/A8
- J3 pad 21: /A11 -> /CPU/A11
- J3 pad 22: /A10 -> /CPU/A10
- J3 pad 23: /A13 -> /CPU/A13
- J3 pad 24: /A12 -> /CPU/A12
- J3 pad 25: /A15 -> /CPU/A15
- J3 pad 26: /A14 -> /CPU/A14
- U1 pad 2: /CPU/AD14 -> /CPU/A14
- U1 pad 3: /CPU/AD13 -> /CPU/A13
- U1 pad 39: /CPU/AD15 -> /CPU/A15
- U1 pad 4: /CPU/AD12 -> /CPU/A12
- U1 pad 5: /CPU/AD11 -> /CPU/A11
- U1 pad 6: /CPU/AD10 -> /CPU/A10
- U1 pad 7: /CPU/AD9 -> /CPU/A9
- U1 pad 8: /CPU/AD8 -> /CPU/A8
- U11 pad 1: /IO_DECODER/LED_PANEL_CS -> /IOWC
- U11 pad 10: /IOWC -> GND
- U11 pad 11: unconnected-(U11-Pad11) -> Net-(U10-Cp)
- U11 pad 12: GND -> Net-(U11-Pad12)
- U11 pad 13: GND -> Net-(U11-Pad13)
- U11 pad 2: /IO_DECODER/LED_PANEL_CS -> /IOWC
- U11 pad 3: Net-(U11-Pad3) -> Net-(U11-Pad12)
- U11 pad 4: Net-(U11-Pad3) -> /IO_DECODER/LED_PANEL_CS
- U11 pad 5: Net-(U11-Pad5) -> /IO_DECODER/LED_PANEL_CS
- U11 pad 6: Net-(U10-Cp) -> Net-(U11-Pad13)
- U11 pad 8: Net-(U11-Pad5) -> unconnected-(U11-Pad8)
- U11 pad 9: /IOWC -> GND
- U13 pad 1: /A14 -> /CPU/A14
- U13 pad 2: /A12 -> /CPU/A12
- U13 pad 21: /A10 -> /CPU/A10
- U13 pad 23: /A11 -> /CPU/A11
- U13 pad 24: /A9 -> /CPU/A9
- U13 pad 25: /A8 -> /CPU/A8
- U13 pad 26: /A13 -> /CPU/A13
- U15 pad 1: Net-(U6-DEN) -> /IOWC
- U15 pad 10: /IOWC -> Net-(U6-DEN)
- U15 pad 11: /MEM_DEC_EN -> unconnected-(U15-Pad11)
- U15 pad 12: /MRDC -> GND
- U15 pad 13: /MWTC -> GND
- U15 pad 2: Net-(U6-DEN) -> /IORC
- U15 pad 3: /CPU/DEN -> /IO_DEC_EN
- U15 pad 4: GND -> /MRDC
- U15 pad 5: GND -> /MWTC
- U15 pad 6: unconnected-(U15-Pad6) -> /MEM_DEC_EN
- U15 pad 8: /IO_DEC_EN -> /CPU/DEN
- U15 pad 9: /IORC -> Net-(U6-DEN)
- U8 pad 1: /A14 -> /CPU/A14
- U8 pad 2: /A12 -> /CPU/A12
- U8 pad 21: /A10 -> /CPU/A10
- U8 pad 23: /A11 -> /CPU/A11
- U8 pad 24: /A9 -> /CPU/A9
- U8 pad 25: /A8 -> /CPU/A8
- U8 pad 26: /A13 -> /CPU/A13
- U9 pad 1: /A14 -> /CPU/A14
- U9 pad 2: /A12 -> /CPU/A12
- U9 pad 21: /A10 -> /CPU/A10
- U9 pad 23: /A11 -> /CPU/A11
- U9 pad 24: /A9 -> /CPU/A9
- U9 pad 25: /A8 -> /CPU/A8
- U9 pad 26: /A13 -> /CPU/A13
Routing:
- net /A9: track 377.5 -> 0.00 mm, vias 4 -> 0
- net /CPU/A11: track 0.00 -> 374.5 mm, vias 0 -> 8
- net /CPU/A13: track 0.00 -> 352.3 mm, vias 0 -> 5
- net /CPU/A14: track 0.00 -> 303.1 mm, vias 0 -> 6
- net /A10: track 277.8 -> 0.00 mm, vias 2 -> 0
- net /CPU/A9: track 0.00 -> 266.9 mm, vias 0 -> 3
- net /A11: track 260.3 -> 0.00 mm, vias 5 -> 0
- net /A8: track 255.7 -> 0.00 mm, vias 4 -> 0
- net /CPU/A10: track 0.00 -> 253.0 mm, vias 0 -> 2
- net /CPU/A12: track 0.00 -> 247.6 mm, vias 0 -> 4
- net /A13: track 245.2 -> 0.00 mm, vias 3 -> 0
- net /CPU/A8: track 0.00 -> 237.2 mm, vias 0 -> 1
- net /A12: track 224.6 -> 0.00 mm, vias 2 -> 0
- net /A14: track 201.4 -> 0.00 mm, vias 1 -> 0
- net /CPU/A15: track 0.00 -> 158.5 mm, vias 0 -> 2
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Other:
- board text added: "PWR"
- board text removed: "PWD"

Commit message: Update 8086-mainboard scheme
Connections:
- net /CPU/A0 renamed /A0
- net /CPU/A1 renamed /A1
- net /CPU/A10 renamed /A10
- net /CPU/A11 renamed /A11
- net /CPU/A12 renamed /A12
- net /CPU/A13 renamed /A13
- net /CPU/A14 renamed /A14
- net /CPU/A15 renamed /A15
- net /CPU/A16 renamed /A16
- net /CPU/A17 renamed /A17
- net /CPU/A18 renamed /A18
- net /CPU/A19 renamed /A19
- net /CPU/A2 renamed /A2
- net /CPU/A3 renamed /A3
- net /CPU/A4 renamed /A4
- net /CPU/A5 renamed /A5
- net /CPU/A6 renamed /A6
- net /CPU/A7 renamed /A7
- net /CPU/A8 renamed /A8
- net /CPU/A9 renamed /A9
- net /CPU/D0 renamed /D0
- net /CPU/D1 renamed /D1
- net /CPU/D2 renamed /D2
- net /CPU/D3 renamed /D3
- net /CPU/D4 renamed /D4
- net /CPU/D5 renamed /D5
- net /CPU/D6 renamed /D6
- net /CPU/D7 renamed /D7

Commit message: Update 8086-mainboard scheme
Parts:
- added JP1: Jumper_2_Open, Connector_PinHeader_2.54mm:PinHeader_1x02_P2.54mm_Vertical, F.Cu at (67.2, 44.0)
- moved H2 1.00 mm to (179.0, 25.0)
- moved H4 1.00 mm to (179.0, 152.0)
- moved R2 0.95 mm to (62.8, 31.7)
- moved C14 0.95 mm to (33.8, 99.2)
- moved C15 0.95 mm to (67.9, 99.2)
- moved C18 0.95 mm to (103.9, 94.3)
- moved C7 0.95 mm to (103.9, 71.7)
- moved D10 0.95 mm to (36.0, 91.0)
- moved J3 0.95 mm to (37.7, 149.4)
- moved R10 0.95 mm to (52.1, 73.7)
- moved R11 0.95 mm to (49.0, 73.7)
- moved R12 0.95 mm to (46.0, 73.7)
- moved R13 0.95 mm to (42.9, 73.7)
- moved R14 0.95 mm to (39.9, 73.7)
- moved R15 0.95 mm to (36.8, 73.7)
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Routing:
- net Net-(JP1-A): track 26.5 -> 34.3 mm
- net /IO_DEC_EN: track 68.3 -> 65.2 mm
- net /A6: track 299.0 -> 296.3 mm
- net /A1: track 301.6 -> 299.9 mm
- net /A3: track 274.6 -> 273.3 mm
- net /A7: track 316.8 -> 315.6 mm
- net /A5: track 288.0 -> 286.7 mm
Other:
- board size 163 x 137 mm -> 164 x 137 mm
- board text added: "CPU"
- board text added: "WAIT"
- board text removed: "8088 CPU"

Commit message: Update 8088-mainboard schematics
Parts:
- removed C14, C15, C19, C9: 100nF, Capacitor_THT:C_Disc_D5.0mm_W2.5mm_P5.00mm
- removed D10: LED7, LED_THT:LED_D3.0mm
- removed D3: LED0, LED_THT:LED_D3.0mm
- removed D4: LED1, LED_THT:LED_D3.0mm
- removed D5: LED2, LED_THT:LED_D3.0mm
- removed D6: LED3, LED_THT:LED_D3.0mm
- removed D7: LED4, LED_THT:LED_D3.0mm
- removed D8: LED5, LED_THT:LED_D3.0mm
- removed D9: LED6, LED_THT:LED_D3.0mm
- removed R10, R11, R12, R13, R14, R15, R16, R9: 680, Resistor_THT:R_Axial_DIN0207_L6.3mm_D2.5mm_P7.62mm_Horizontal
- removed U10: 74LS273, Package_DIP:DIP-20_W7.62mm
- removed U11, U15: 74LS00, Package_DIP:DIP-14_W7.62mm
- removed U6: 8288, Package_DIP:DIP-20_W7.62mm
- U1: value 8088_Max_Mode -> 8088_Min_Mode
- moved U12 54.6 mm to (105.9, 112.1)
- moved C16 54.5 mm to (100.3, 104.5)
- moved U7 53.5 mm to (105.9, 93.9)
- moved C10 53.4 mm to (100.3, 86.3)
- moved U14 49.3 mm to (105.8, 57.5)
- moved C18 44.6 mm to (100.2, 49.9), turned to -90 degrees
- moved J3 39.6 mm to (37.7, 109.9)
- moved H4 39.2 mm to (175.0, 113.0)
- moved H3 39.0 mm to (25.0, 113.0)
- moved J2 38.1 mm to (37.7, 88.5)
- moved U3 22.6 mm to (105.7, 39.3)
- moved J_DEBUG1 17.9 mm to (105.7, 26.5)
- moved C6 17.9 mm to (100.1, 31.6), turned to -90 degrees
- moved C17 9.03 mm to (134.2, 88.8)
- moved U13 9.03 mm to (139.8, 104.1)
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Connections:
- J2 pad 10: /D0 -> /A12
- J2 pad 11: /A1 -> /A11
- J2 pad 12: /A0 -> /A10
- J2 pad 13: /A3 -> /A9
- J2 pad 14: /A2 -> /A8
- J2 pad 15: /A5 -> /A7
- J2 pad 16: /A4 -> /A6
- J2 pad 17: /A7 -> /A5
- J2 pad 18: /A6 -> /A4
- J2 pad 19: /A9 -> /A3
- J2 pad 20: /A8 -> /A2
- J2 pad 21: /A11 -> /A1
- J2 pad 22: /A10 -> /A0
- J2 pad 23: /A13 -> /D7
- J2 pad 24: /A12 -> /D6
- J2 pad 25: /A15 -> /D5
- J2 pad 26: /A14 -> /D4
- J2 pad 27: /A17 -> /D3
- J2 pad 28: /A16 -> /D2
- J2 pad 29: /A19 -> /D1
- J2 pad 3: /D7 -> /A19
- J2 pad 30: /A18 -> /D0
- J2 pad 31: /IORC -> /IOM
- J2 pad 32: /IOWC -> /RD
- J2 pad 33: /MRDC -> /WR
- J2 pad 34: /MWTC -> unconnected-(J2-Pin_34-Pad34)
- J2 pad 4: /D6 -> /A18
- J2 pad 5: /D5 -> /A17
- J2 pad 6: /D4 -> /A16
- J2 pad 7: /D3 -> /A15
- J2 pad 8: /D2 -> /A14
- J2 pad 9: /D1 -> /A13
- J3 pad 10: /D0 -> /A12
- J3 pad 11: /A1 -> /A11
- J3 pad 12: /A0 -> /A10
- J3 pad 13: /A3 -> /A9
- J3 pad 14: /A2 -> /A8
- J3 pad 15: /A5 -> /A7
- J3 pad 16: /A4 -> /A6
- J3 pad 17: /A7 -> /A5
- J3 pad 18: /A6 -> /A4
- J3 pad 19: /A9 -> /A3
- J3 pad 20: /A8 -> /A2
- J3 pad 21: /A11 -> /A1
- J3 pad 22: /A10 -> /A0
- J3 pad 23: /A13 -> /D7
- J3 pad 24: /A12 -> /D6
- J3 pad 25: /A15 -> /D5
- J3 pad 26: /A14 -> /D4
- J3 pad 27: /A17 -> /D3
- J3 pad 28: /A16 -> /D2
- J3 pad 29: /A19 -> /D1
- J3 pad 3: /D7 -> /A19
- J3 pad 30: /A18 -> /D0
- J3 pad 31: /IORC -> /IOM
- J3 pad 32: /IOWC -> /RD
- J3 pad 33: /MRDC -> /WR
- J3 pad 34: /MWTC -> unconnected-(J3-Pin_34-Pad34)
- J3 pad 4: /D6 -> /A18
- J3 pad 5: /D5 -> /A17
- J3 pad 6: /D4 -> /A16
- J3 pad 7: /D3 -> /A15
- J3 pad 8: /D2 -> /A14
- J3 pad 9: /D1 -> /A13
- J_DEBUG1 pad 6: /MRDC -> /IOM
- J_DEBUG1 pad 7: /MWTC -> /WR
- J_DEBUG1 pad 8: /IORC -> /RD
- J_DEBUG1 pad 9: /IOWC -> /CPU/DT_R
- U1 pad 25: unconnected-(U1-QS0-Pad25) -> /ALE
- U1 pad 26: /CPU/S0 -> /CPU/DEN
- U1 pad 27: /CPU/S1 -> /CPU/DT_R
- U1 pad 28: /CPU/S2 -> /IOM
- U1 pad 29: unconnected-(U1-~{LOCK}-Pad29) -> /WR
- U1 pad 31: unconnected-(U1-~{RQ}/~{GT0}-Pad31) -> GND
- U1 pad 32: unconnected-(U1-~{RD}-Pad32) -> /RD
- U1 pad 33: GND -> VCC
- U12 pad 15: /IO_DECODER/LED_PANEL_CS -> unconnected-(U12-O0-Pad15)
- U12 pad 6: /IO_DEC_EN -> /IOM
- U13 pad 22: /MRDC -> /RD
- U13 pad 27: /MWTC -> /WR
- U7 pad 4: GND -> /IOM
- U7 pad 6: /MEM_DEC_EN -> VCC
- U8 pad 22: /MRDC -> /RD
- U9 pad 22: /MRDC -> /RD
- U9 pad 27: /MWTC -> /WR
Routing:
- net VCC: track 606.6 -> 0.00 mm, vias 2 -> 0
- net /A11: track 374.5 -> 0.00 mm, vias 8 -> 0
- net /A13: track 352.3 -> 0.00 mm, vias 5 -> 0
- net /A7: track 315.6 -> 0.00 mm, vias 4 -> 0
- net /A14: track 303.1 -> 0.00 mm, vias 6 -> 0
- net /A1: track 299.9 -> 0.00 mm, vias 5 -> 0
- net /A6: track 296.3 -> 0.00 mm, vias 4 -> 0
- net /D6: track 292.7 -> 0.00 mm, vias 3 -> 0
- net /D7: track 291.5 -> 0.00 mm, vias 3 -> 0
- net /A5: track 286.7 -> 0.00 mm, vias 2 -> 0
- net /A0: track 279.6 -> 0.00 mm, vias 2 -> 0
- net /A3: track 273.3 -> 0.00 mm, vias 5 -> 0
- net /D1: track 267.1 -> 0.00 mm, vias 9 -> 0
- net /A9: track 266.9 -> 0.00 mm, vias 3 -> 0
- net /D4: track 264.6 -> 0.00 mm, vias 5 -> 0
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Other:
- board size 164 x 137 mm -> 160 x 98 mm
- board text added: "DT_R"
- board text added: "IOM"
- board text added: "RD"
- board text added: "WR"
- board text removed: "DEBUG LEDs"
- board text removed: "IORC"
- board text removed: "IOWC"
- board text removed: "MRDC"
- board text removed: "MWTC"

Commit message: Finalize 8088 mainboard rev1.0 for production
Parts:
- removed C17: 100nF, Capacitor_THT:C_Disc_D5.0mm_W2.5mm_P5.00mm
- removed the C4 at (51.8, 36.5)
- removed JP1: Jumper_2_Open, Connector_PinHeader_2.54mm:PinHeader_1x02_P2.54mm_Vertical
- removed J_DEBUG1: DEBUG, Connector_PinHeader_2.54mm:PinHeader_1x10_P2.54mm_Vertical
- removed U13: HM62256BLP, Package_DIP:DIP-28_W15.24mm
- added C5: 10 uF, Capacitor_THT:CP_Radial_D4.0mm_P1.50mm, F.Cu at (53.7, 30.0)
- added D3: BAT85, Diode_THT:D_DO-35_SOD27_P7.62mm_Horizontal, F.Cu at (174.8, 40.7)
- added D4: BAT85, Diode_THT:D_DO-35_SOD27_P7.62mm_Horizontal, F.Cu at (180.5, 48.3)
- added J1: Conn_01x10, Connector_PinHeader_2.54mm:PinHeader_1x10_P2.54mm_Vertical, F.Cu at (117.7, 29.2)
- added J5: Ext CLK, Connector_PinHeader_2.54mm:PinHeader_1x02_P2.54mm_Vertical, F.Cu at (175.3, 30.9)
- added Q1: NDP6020P, Package_TO_SOT_THT:TO-220-3_Horizontal_TabDown, F.Cu at (25.2, 60.9)
- added R5: 10k, Resistor_THT:R_Axial_DIN0207_L6.3mm_D2.5mm_P7.62mm_Horizontal, F.Cu at (44.3, 47.2)
- added R6: 1k, Resistor_THT:R_Axial_DIN0207_L6.3mm_D2.5mm_P7.62mm_Horizontal, F.Cu at (177.6, 48.3)
- added R8: 10k, Resistor_THT:R_Axial_DIN0207_L6.3mm_D2.5mm_P7.62mm_Horizontal, F.Cu at (59.7, 39.5)
- added R9: 10k, Resistor_THT:R_Axial_DIN0207_L6.3mm_D2.5mm_P7.62mm_Horizontal, F.Cu at (62.8, 47.2)
- added SW2: SW_DIP_x02, Button_Switch_THT:SW_DIP_SPSTx02_Slide_9.78x7.26mm_W7.62mm_P2.54mm, F.Cu at (160.7, 36.9)
- C13: value 410 uF -> 220 uF; footprint Capacitor_THT:CP_Radial_D8.0mm_P3.50mm -> Capacitor_THT:CP_Radial_D5.0mm_P2.00mm
- R3: renamed from R4; value 330 -> 680
- R4: renamed from R3; value 330 -> 2k
- U1: footprint Package_DIP:DIP-40_W15.24mm -> Package_DIP:DIP-40_W15.24mm_Socket
- U2: renamed from U3; footprint Package_DIP:DIP-20_W7.62mm -> Package_DIP:DIP-20_W7.62mm_Socket
- U3: renamed from U14; footprint Package_DIP:DIP-20_W7.62mm -> Package_DIP:DIP-20_W7.62mm_Socket
- U4: renamed from U5; footprint Package_DIP:DIP-20_W7.62mm -> Package_DIP:DIP-20_W7.62mm_Socket
- U5: renamed from U2; footprint Package_DIP:DIP-18_W7.62mm -> Package_DIP:DIP-18_W7.62mm_Socket
- U6: renamed from U7; footprint Package_DIP:DIP-16_W7.62mm -> Package_DIP:DIP-16_W7.62mm_Socket
- U7: renamed from U12; footprint Package_DIP:DIP-16_W7.62mm -> Package_DIP:DIP-16_W7.62mm_Socket
- U8: footprint Package_DIP:DIP-28_W15.24mm -> Socket:DIP_Socket-28_W11.9mm_W12.7mm_W15.24mm_W17.78mm_W18.5mm_3M_228-1277-00-0602J
- U9: footprint Package_DIP:DIP-28_W15.24mm -> Package_DIP:DIP-28_W15.24mm_Socket
- moved SW1 146.7 mm to (28.6, 85.3), turned to -90 degrees
- moved U8 111.5 mm to (57.1, 132.4)
- moved C11 103.4 mm to (57.1, 111.2), turned to 180 degrees
- moved J3 85.2 mm to (119.5, 133.5)
- moved J2 84.2 mm to (119.5, 108.1)
- moved U9 79.8 mm to (62.6, 101.1)
- moved C12 77.4 mm to (59.5, 85.8)
- moved C9 65.9 mm to (159.5, 57.4)
- moved C10 65.1 mm to (159.8, 78.2)
- moved U6 63.7 mm to (162.7, 65.0)
- moved U7 62.8 mm to (163.0, 85.9)
- moved C3 31.8 mm to (114.6, 78.2)
- moved U3 30.8 mm to (117.7, 85.9)
- moved H4 28.8 mm to (185.0, 140.0)
- moved H3 27.0 mm to (25.0, 140.0)
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- renumbered C8 to C1, C16 to C10, C6 to C2, C18 to C3, C7 to C4, C3 to C6, C1 to C7, C2 to C8, C10 to C9, J1 to J4
Connections:
- J2 pad 34: unconnected-(J2-Pin_34-Pad34) -> /RDY
- J2 pad 37: GND -> /EXPANSION_CONNECTOR/MEM_EXP0_CS
- J2 pad 38: /CLK -> /EXPANSION_CONNECTOR/IO_EXP0_CS
- J2 pad 39: /EXPANSION_CONNECTOR/IO_EXP0_CS -> GND
- J2 pad 40: /EXPANSION_CONNECTOR/MEM_EXP0_CS -> /CLK
- J3 pad 34: unconnected-(J3-Pin_34-Pad34) -> /RDY
- J3 pad 37: GND -> /EXPANSION_CONNECTOR/MEM_EXP1_CS
- J3 pad 38: /CLK -> /EXPANSION_CONNECTOR/IO_EXP1_CS
- J3 pad 39: /EXPANSION_CONNECTOR/IO_EXP1_CS -> GND
- J3 pad 40: /EXPANSION_CONNECTOR/MEM_EXP1_CS -> /CLK
- J4 pad 1: VCC -> Net-(J4-Pin_1)
- R2 pad 2: Net-(JP1-A) -> /RDY
- U5 pad 1: unconnected-(U2-CSYNC-Pad1) -> GND
- U5 pad 13: GND -> Net-(U5-F/~{C})
- U5 pad 14: GND -> Net-(D3-A)
- U5 pad 4: Net-(JP1-A) -> /RDY
- U5 pad 6: Net-(JP1-A) -> /RDY
- U6 pad 14: /MEM_DECODER/RAM_BANK1_CS -> unconnected-(U6-O1-Pad14)
Routing:
- net VCC: track 0.00 -> 540.3 mm, vias 0 -> 4
- net /A6: track 0.00 -> 310.1 mm, vias 0 -> 6
- net /A7: track 0.00 -> 307.1 mm, vias 0 -> 7
- net /RD: track 0.00 -> 277.5 mm, vias 0 -> 1
- net /RESET: track 0.00 -> 264.0 mm, vias 0 -> 3
- net /WR: track 0.00 -> 249.4 mm, vias 0 -> 3
- net /A5: track 0.00 -> 245.0 mm, vias 0 -> 4
- net /A4: track 0.00 -> 232.5 mm, vias 0 -> 1
- net /A1: track 0.00 -> 230.4 mm, vias 0 -> 2
- net /CLK: track 0.00 -> 225.8 mm, vias 0 -> 3
- net /A3: track 0.00 -> 224.2 mm, vias 0 -> 6
- net /RDY: track 0.00 -> 220.9 mm
- net /A2: track 0.00 -> 214.4 mm, vias 0 -> 4
- net /A0: track 0.00 -> 214.2 mm, vias 0 -> 7
- net /IOM: track 0.00 -> 214.1 mm, vias 0 -> 2
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Other:
- board size 160 x 98 mm -> 170 x 125 mm
- board text added: "+5V"
- board text added: "2026"
- board text added: "8088"
- board text added: "DT/R"
- board text added: "EFI"
- board text added: "EXP0"
- board text added: "EXP1"
- board text added: "EXT CLK INPUT 0-5 V"
- board text added: "Homebrew Computer"
- board text added: "IO/M"
- board text added: "Source: github.com/i-melnichenko/8088-homebrew-computer"
- board text added: "~DEN"
- board text added: "~RD"
- board text added: "~WR"
- board text removed: "+5v"
- board text removed: "8088 Mainboard"
- board text removed: "DEN"
- board text removed: "DT_R"
- board text removed: "EXT0"
- board text removed: "EXT1"
- board text removed: "IOM"
- board text removed: "Project: github.com/i-melnichenko/8088-homebrew-computer"
- board text removed: "RAM BANK1"
- board text removed: "RD"
- board text removed: "RES"
- board text removed: "WR"
