File: hardware/kicad/8088-mainboard/MEM_DECODER.kicad_sch (KiCad schematic)
At the start: 2 parts, among them U7 74LS138

Commit message: Add PSB board design
Connections:
- net MEM_EXP2_CS renamed MEM_C0000_DFFFF
Changed lines of the file:
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@@
-	(wire
-		(pts
-			(xy 134.62 73.66) (xy 154.94 73.66)
-		)
-		(stroke
-			(width 0)
-			(type default)
-		)
-	)
 	(wire
 		(pts
@@
 		)
 	)
-	(label "MEM_C0000_DFFFF"
-		(at 134.62 73.66 0)
-		(effects
-			(font
-				(size 1.27 1.27)
-			)
-			(justify left bottom)
-		)
-	)
 	(label "MEM_60000_7FFFF"
 		(at 119.38 66.04 180)
@@
 		(effects
 			(font
-				(size 1.27 1.27)
-			)
-			(justify left)
-		)
-	)
-	(hierarchical_label "MEM_EXP2_CS"
-		(shape input)
-		(at 154.94 73.66 0)
-		(effects
-			(font

Commit message: Update 8088-mainboard schematics for refined connections and label adjustments
Connections:
- net VCC: no longer U7.6 (E3)
- net A0 renamed A17
- net A1 renamed A18
- net A2 renamed A19
- net MEM_40000_5FFFF: no longer names the net of U7.13 (O2)
- net MEM_60000_7FFFF: no longer names the net of U7.12 (O3)
- net MEM_C0000_DFFFF: no longer names the net of U7.9 (O6)
- new net MEM_DEC_EN: U7.6 (E3)
- no-connect marks 0 -> 3
Other:
- note added: "MEM_00000_1FFFF"
- note added: "MEM_20000_3FFFF"
- note added: "MEM_40000_5FFFF"
- note added: "MEM_60000_7FFFF"
- note added: "MEM_80000_9FFFF"
- note added: "MEM_A0000_BFFFF"
- note added: "MEM_C0000_DFFFF"
- note added: "MEM_E0000_FFFFF"

Commit message: Update 8086-mainboard scheme
Changed lines of the file:
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@@
+		)
+	)
+	(bus
+		(pts
+			(xy 0.1524 35.7124) (xy 26.8224 35.7124)
+		)
+		(stroke
+			(width 0)
+			(type default)
 		)
 	)
@@
 		)
 	)
+	(bus
+		(pts
+			(xy 0.1524 0.1524) (xy 36.9824 0.1524)
+		)
+		(stroke
+			(width 0)
+			(type default)
+		)
+	)
 	(wire
 		(pts
 			(xy 121.92 71.12) (xy 101.6 71.12)
+		)
+		(stroke
+			(width 0)
+			(type default)
+		)
+	)
+	(bus
+		(pts
+			(xy 0.1524 0.1524) (xy 0.1524 35.7124)
 		)
 		(stroke
@@
 	)
 	(hierarchical_label "RAM_BANK1_CS"
-		(shape input)
+		(shape output)
 		(at 121.92 60.96 0)
 		(effects
@@
 	)
 	(hierarchical_label "MEM_EXP1_CS"
-		(shape input)
+		(shape output)
 		(at 121.92 71.12 0)
 		(effects
@@
 	)
 	(hierarchical_label "ROM_CS"
-		(shape input)
+		(shape output)
 		(at 121.92 76.2 0)
 		(effects
@@
 	)
 	(hierarchical_label "RAM_BANK0_CS"
-		(shape input)
+		(shape output)
 		(at 121.92 58.42 0)
 		(effects
@@
 	)
 	(hierarchical_label "MEM_EXP0_CS"
-		(shape input)
+		(shape output)
 		(at 121.92 68.58 0)
 		(effects

Commit message: Update 8086-mainboard scheme
Changed lines of the file:
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@@
-		)
-	)
-	(bus
-		(pts
-			(xy 0.1524 35.7124) (xy 26.8224 35.7124)
-		)
-		(stroke
-			(width 0)
-			(type default)
 		)
 	)
@@
 		)
 	)
-	(bus
-		(pts
-			(xy 0.1524 0.1524) (xy 36.9824 0.1524)
-		)
-		(stroke
-			(width 0)
-			(type default)
-		)
-	)
 	(wire
 		(pts
@@
 		)
 		(stroke
-			(width 0)
-			(type default)
-		)
-	)
-	(bus
-		(pts
-			(xy 0.1524 0.1524) (xy 0.1524 35.7124)
-		)
-		(stroke

Commit message: Update 8088-mainboard schematics
Connections:
- net MEM_DEC_EN is gone; now on net VCC: U7.6 (E3)
- net GND: no longer U7.4 (E1)
- new net IOM: U7.4 (E1)
Changed lines of the file:
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@@
+	(wire
+		(pts
+			(xy 63.5 71.12) (xy 76.2 71.12)
+		)
+		(stroke
+			(width 0)
+			(type default)
+		)
+	)
 	(wire
 		(pts
@@
 			(width 0)
 			(type default)
-		)
-	)
-	(hierarchical_label "MEM_DEC_EN"
-		(shape input)
-		(at 76.2 71.12 180)
-		(effects
-			(font
-				(size 1.27 1.27)
-			)
-			(justify right)
 		)
 	)
@@
 			)
 			(justify left)
+		)
+	)
+	(hierarchical_label "IOM"
+		(shape input)
+		(at 76.2 76.2 180)
+		(effects
+			(font
+				(size 1.27 1.27)
+			)
+			(justify right)
 		)
 	)
@@
 	)
 	(symbol
-		(lib_id "power:GND")
-		(at 76.2 76.2 270)
+		(lib_id "power:VCC")
+		(at 63.5 71.12 0)
 		(unit 1)
 		(body_style 1)
@@
 		(in_pos_files yes)
 		(dnp no)
-		(fields_autoplaced yes)
-		(property "Reference" "#PWR041"
-			(at 69.85 76.2 0)
-			(hide yes)
-			(show_name no)
-			(do_not_autoplace no)
-			(effects
-				(font
-					(size 1.27 1.27)
-				)
-			)
-		)
-		(property "Value" "GND"
-			(at 72.39 76.1999 90)
-			(show_name no)
-			(do_not_autoplace no)
-			(effects
-				(font
-					(size 1.27 1.27)
-				)
-				(justify right)
+		(property "Reference" "#PWR039"
+			(at 63.5 74.93 0)
+			(hide yes)
+			(show_name no)
+			(do_not_autoplace no)
+			(effects
+				(font
+					(size 1.27 1.27)
+				)
+			)
+		)
+		(property "Value" "VCC"
+			(at 63.5 68.072 90)
+			(show_name no)
+			(do_not_autoplace no)
+			(effects
+				(font
+					(size 1.27 1.27)
+				)
+				(justify left)
 			)
 		)
 		(property "Footprint" ""
-			(at 76.2 76.2 0)
+			(at 63.5 71.12 0)
 			(hide yes)
 			(show_name no)
@@
 		)
 		(property "Datasheet" ""
-			(at 76.2 76.2 0)
-			(hide yes)
-			(show_name no)
-			(do_not_autoplace no)
-			(effects
-				(font
-					(size 1.27 1.27)
-				)
-			)
-		)
-		(property "Description" "Power symbol creates a global label with name \"GND\" , ground"
-			(at 76.2 76.2 0)
+			(at 63.5 71.12 0)
+			(hide yes)
+			(show_name no)
+			(do_not_autoplace no)
+			(effects
+				(font
+					(size 1.27 1.27)
+				)
+			)
+		)
+		(property "Description" "Power symbol creates a global label with name \"VCC\""
+			(at 63.5 71.12 0)
 			(hide yes)
 			(show_name no)
@@
 			(project "8088-mainboard"
 				(path "/15ce4f45-6f32-456e-874c-aac11293789a/8603fecf-1343-4cbc-8a43-8cc8a41e8f5f"
-					(reference "#PWR041")
+					(reference "#PWR039")
 					(unit 1)
 				)

Commit message: Finalize 8088 mainboard rev1.0 for production
Parts:
- U6: renamed from U7; footprint Package_DIP:DIP-16_W7.62mm -> Package_DIP:DIP-16_W7.62mm_Socket
- renumbered C10 to C9
Connections:
- net RAM_BANK1_CS: no longer names the net of U6.14 (O1)
- no-connect marks 3 -> 4
Changed lines of the file:
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@@
 		(at 121.92 66.04)
+	)
+	(no_connect
+		(at 121.92 60.96)
 	)
 	(wire
@@
 			)
 			(justify right)
-		)
-	)
-	(hierarchical_label "RAM_BANK1_CS"
-		(shape output)
-		(at 121.92 60.96 0)
-		(effects
-			(font
-				(size 1.27 1.27)
-			)
-			(justify left)
 		)
 	)
@@
 		(in_pos_files yes)
 		(dnp no)
-		(property "Reference" "C10"
+		(property "Reference" "C9"
 			(at 81.28 40.894 0)
 			(show_name no)
@@
 			(project "8088-mainboard"
 				(path "/15ce4f45-6f32-456e-874c-aac11293789a/8603fecf-1343-4cbc-8a43-8cc8a41e8f5f"
-					(reference "C10")
+					(reference "C9")
 					(unit 1)
 				)
@@
 		(dnp no)
 		(fields_autoplaced yes)
-		(property "Reference" "#PWR040"
+		(property "Reference" "#PWR034"
 			(at 69.85 73.66 0)
 			(hide yes)
@@
 			(project "8088-mainboard"
 				(path "/15ce4f45-6f32-456e-874c-aac11293789a/8603fecf-1343-4cbc-8a43-8cc8a41e8f5f"
-					(reference "#PWR040")
+					(reference "#PWR034")
 					(unit 1)
 				)
@@
 		(in_pos_files yes)
 		(dnp no)
-		(property "Reference" "#PWR039"
+		(property "Reference" "#PWR033"
 			(at 63.5 74.93 0)
 			(hide yes)
@@
 			(project "8088-mainboard"
 				(path "/15ce4f45-6f32-456e-874c-aac11293789a/8603fecf-1343-4cbc-8a43-8cc8a41e8f5f"
-					(reference "#PWR039")
+					(reference "#PWR033")
 					(unit 1)
 				)
@@
 		(in_pos_files yes)
 		(dnp no)
-		(property "Reference" "#PWR037"
+		(property "Reference" "#PWR036"
 			(at 88.9 45.72 0)
 			(hide yes)
@@
 			(project "8088-mainboard"
 				(path "/15ce4f45-6f32-456e-874c-aac11293789a/8603fecf-1343-4cbc-8a43-8cc8a41e8f5f"
-					(reference "#PWR037")
+					(reference "#PWR036")
 					(unit 1)
 				)
@@
 		(dnp no)
 		(fields_autoplaced yes)
-		(property "Reference" "#PWR038"
+		(property "Reference" "#PWR035"
 			(at 71.12 46.99 0)
 			(hide yes)
@@
 			(project "8088-mainboard"
 				(path "/15ce4f45-6f32-456e-874c-aac11293789a/8603fecf-1343-4cbc-8a43-8cc8a41e8f5f"
-					(reference "#PWR038")
+					(reference "#PWR035")
 					(unit 1)
 				)
@@
 		(dnp no)
 		(fields_autoplaced yes)
-		(property "Reference" "#PWR036"
+		(property "Reference" "#PWR037"
 			(at 88.9 90.17 0)
 			(hide yes)
@@
 			(project "8088-mainboard"
 				(path "/15ce4f45-6f32-456e-874c-aac11293789a/8603fecf-1343-4cbc-8a43-8cc8a41e8f5f"
-					(reference "#PWR036")
+					(reference "#PWR037")
 					(unit 1)
 				)
@@
 		(in_pos_files yes)
 		(dnp no)
-		(property "Reference" "U7"
+		(property "Reference" "U6"
 			(at 90.932 51.054 0)
 			(show_name no)
@@
 			)
 		)
-		(property "Footprint" "Package_DIP:DIP-16_W7.62mm"
+		(property "Footprint" "Package_DIP:DIP-16_W7.62mm_Socket"
 			(at 88.9 66.04 0)
 			(hide yes)
@@
 			(project "8088-mainboard"
 				(path "/15ce4f45-6f32-456e-874c-aac11293789a/8603fecf-1343-4cbc-8a43-8cc8a41e8f5f"
-					(reference "U7")
+					(reference "U6")
 					(unit 1)
 				)
