File: hardware/kicad/8088-mainboard/RAM.kicad_sch (KiCad schematic)
At the start: 4 parts, among them U13 HM62256BLP, U9 HM62256BLP

Commit message: Update 8086-mainboard scheme
Other:
- moved on the sheet: C17, U13

Commit message: Update 8088-mainboard schematics
Connections:
- net MRDC renamed RD
- net MWTC renamed WR
Changed lines of the file:
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@@
+		)
+	)
+	(hierarchical_label "WR"
+		(shape input)
+		(at 210.82 104.14 0)
+		(effects
+			(font
+				(size 1.27 1.27)
+			)
+			(justify left)
 		)
 	)
@@
 		)
 	)
-	(hierarchical_label "MRDC"
+	(hierarchical_label "RD"
 		(shape input)
-		(at 210.82 101.6 0)
+		(at 133.35 101.6 0)
 		(effects
 			(font
@@
 		)
 	)
-	(hierarchical_label "MWTC"
-		(shape input)
-		(at 210.82 104.14 0)
-		(effects
-			(font
-				(size 1.27 1.27)
-			)
-			(justify left)
-		)
-	)
-	(hierarchical_label "MWTC"
+	(hierarchical_label "WR"
 		(shape input)
 		(at 133.35 104.14 0)
@@
 		)
 	)
-	(hierarchical_label "MRDC"
+	(hierarchical_label "RD"
 		(shape input)
-		(at 133.35 101.6 0)
+		(at 210.82 101.6 0)
 		(effects
 			(font

Commit message: Finalize 8088 mainboard rev1.0 for production
Parts:
- removed C17: 100nF, Capacitor_THT:C_Disc_D5.0mm_W2.5mm_P5.00mm, symbol Device:C
- removed U13: HM62256BLP, Package_DIP:DIP-28_W15.24mm, symbol Memory_RAM:HM62256BLP
- U9: footprint Package_DIP:DIP-28_W15.24mm -> Package_DIP:DIP-28_W15.24mm_Socket
Other:
- moved on the sheet: C12, U9
