File: hardware/kicad/8088-mainboard/ROM.kicad_sch (KiCad schematic)
At the start: 2 parts, among them U8 28C256

Commit message: Update 8088-mainboard schematics
Connections:
- net MRDC renamed RD
Changed lines of the file:
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@@
-		)
-	)
-	(hierarchical_label "MRDC"
-		(shape input)
-		(at 134.62 115.57 180)
-		(effects
-			(font
-				(size 1.27 1.27)
-			)
-			(justify right)
 		)
 	)
@@
 		)
 	)
+	(hierarchical_label "RD"
+		(shape input)
+		(at 134.62 115.57 180)
+		(effects
+			(font
+				(size 1.27 1.27)
+			)
+			(justify right)
+		)
+	)

Commit message: Finalize 8088 mainboard rev1.0 for production
Parts:
- U8: footprint Package_DIP:DIP-28_W15.24mm -> Socket:DIP_Socket-28_W11.9mm_W12.7mm_W15.24mm_W17.78mm_W18.5mm_3M_228-1277-00-0602J
Changed lines of the file:
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@@
 		(dnp no)
 		(fields_autoplaced yes)
-		(property "Reference" "#PWR042"
+		(property "Reference" "#PWR043"
 			(at 127 63.5 0)
 			(hide yes)
@@
 			(project "8088-mainboard"
 				(path "/15ce4f45-6f32-456e-874c-aac11293789a/ab02926d-0ef6-4450-b8f0-24a52f381100"
-					(reference "#PWR042")
+					(reference "#PWR043")
 					(unit 1)
 				)
@@
 		(dnp no)
 		(fields_autoplaced yes)
-		(property "Reference" "#PWR044"
+		(property "Reference" "#PWR046"
 			(at 144.78 129.54 0)
 			(hide yes)
@@
 			(project "8088-mainboard"
 				(path "/15ce4f45-6f32-456e-874c-aac11293789a/ab02926d-0ef6-4450-b8f0-24a52f381100"
-					(reference "#PWR044")
+					(reference "#PWR046")
 					(unit 1)
 				)
@@
 		(in_pos_files yes)
 		(dnp no)
-		(property "Reference" "#PWR043"
+		(property "Reference" "#PWR045"
 			(at 144.78 62.23 0)
 			(hide yes)
@@
 			(project "8088-mainboard"
 				(path "/15ce4f45-6f32-456e-874c-aac11293789a/ab02926d-0ef6-4450-b8f0-24a52f381100"
-					(reference "#PWR043")
+					(reference "#PWR045")
 					(unit 1)
 				)
@@
 			)
 		)
-		(property "Footprint" "Package_DIP:DIP-28_W15.24mm"
+		(property "Footprint" "Socket:DIP_Socket-28_W11.9mm_W12.7mm_W15.24mm_W17.78mm_W18.5mm_3M_228-1277-00-0602J"
 			(at 144.78 95.25 0)
 			(hide yes)
@@
 		(in_pos_files yes)
 		(dnp no)
-		(property "Reference" "#PWR045"
+		(property "Reference" "#PWR044"
 			(at 138.43 113.03 0)
 			(hide yes)
@@
 			(project "8088-mainboard"
 				(path "/15ce4f45-6f32-456e-874c-aac11293789a/ab02926d-0ef6-4450-b8f0-24a52f381100"
-					(reference "#PWR045")
+					(reference "#PWR044")
 					(unit 1)
 				)
