File: hardware/kicad/8088-mainboard/CLOCK.kicad_sch (KiCad schematic)
At the start: 11 parts, among them SW1 Reset, U2 8284, Y1 14.31818 MHz

Commit message: Update 8088-mainboard schematics for refined connections and label adjustments
Connections:
- net OSC: no longer names the net of U2.12 (OSC)
- net PCLK: no longer names the net of U2.2 (PCLK)
- no-connect marks 1 -> 3
Changed lines of the file:
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@@
 		(at 125.73 100.33)
 	)
+	(no_connect
+		(at 146.05 97.79)
+	)
+	(no_connect
+		(at 146.05 95.25)
+	)
 	(wire
 		(pts
@@
 	(wire
 		(pts
-			(xy 156.21 72.39) (xy 143.51 72.39)
-		)
-		(stroke
-			(width 0)
-			(type default)
-		)
-	)
-	(wire
-		(pts
 			(xy 157.48 118.11) (xy 161.29 118.11)
 		)
@@
 		(pts
 			(xy 123.19 85.09) (xy 123.19 87.63)
-		)
-		(stroke
-			(width 0)
-			(type default)
-		)
-	)
-	(wire
-		(pts
-			(xy 156.21 73.025) (xy 156.21 72.39)
 		)
 		(stroke
@@
 		(shape input)
 		(at 146.05 85.09 0)
-		(effects
-			(font
-				(size 1.27 1.27)
-			)
-			(justify left)
-		)
-	)
-	(hierarchical_label "OSC"
-		(shape input)
-		(at 146.05 97.79 0)
-		(effects
-			(font
-				(size 1.27 1.27)
-			)
-			(justify left)
-		)
-	)
-	(hierarchical_label "PCLK"
-		(shape input)
-		(at 146.05 95.25 0)
 		(effects
 			(font
@@
 	(symbol
 		(lib_id "power:GND")
-		(at 156.21 73.025 0)
+		(at 143.51 72.39 90)
 		(unit 1)
 		(body_style 1)
@@
 		(fields_autoplaced yes)
 		(property "Reference" "#PWR04"
-			(at 156.21 79.375 0)
+			(at 149.86 72.39 0)
 			(hide yes)
 			(show_name no)
@@
 		)
 		(property "Value" "GND"
-			(at 156.21 78.105 0)
-			(show_name no)
-			(do_not_autoplace no)
-			(effects
-				(font
-					(size 1.27 1.27)
-				)
+			(at 147.32 72.3899 90)
+			(show_name no)
+			(do_not_autoplace no)
+			(effects
+				(font
+					(size 1.27 1.27)
+				)
+				(justify right)
 			)
 		)
 		(property "Footprint" ""
-			(at 156.21 73.025 0)
+			(at 143.51 72.39 0)
 			(hide yes)
 			(show_name no)
@@
 		)
 		(property "Datasheet" ""
-			(at 156.21 73.025 0)
+			(at 143.51 72.39 0)
 			(hide yes)
 			(show_name no)
@@
 		)
 		(property "Description" "Power symbol creates a global label with name \"GND\" , ground"
-			(at 156.21 73.025 0)
-			(hide yes)
-			(show_name no)
+			(at 143.51 72.39 0)
+			(hide yes)
+			(show_name no)

Commit message: Update 8086-mainboard scheme
Other:
- moved on the sheet: C2, Y1
Changed lines of the file:
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@@
-	)
-	(junction
-		(at 173.99 118.11)
-		(diameter 0)
-		(color 0 0 0 0)
 	)
 	(junction
@@
 	)
 	(junction
-		(at 157.48 118.11)
+		(at 123.19 92.71)
 		(diameter 0)
 		(color 0 0 0 0)
 	)
 	(junction
-		(at 123.19 92.71)
+		(at 175.26 118.11)
 		(diameter 0)
 		(color 0 0 0 0)
@@
 		(color 0 0 0 0)
 	)
+	(junction
+		(at 157.48 118.11)
+		(diameter 0)
+		(color 0 0 0 0)
+	)
 	(no_connect
 		(at 125.73 100.33)
@@
 	(wire
 		(pts
-			(xy 168.91 118.11) (xy 173.99 118.11)
+			(xy 170.18 118.11) (xy 175.26 118.11)
 		)
 		(stroke
@@
 	(wire
 		(pts
-			(xy 157.48 118.11) (xy 161.29 118.11)
+			(xy 157.48 118.11) (xy 162.56 118.11)
 		)
 		(stroke
@@
 	(wire
 		(pts
-			(xy 173.99 105.41) (xy 173.99 118.11)
+			(xy 175.26 105.41) (xy 175.26 118.11)
 		)
 		(stroke
@@
 	(wire
 		(pts
-			(xy 173.99 118.11) (xy 173.99 121.92)
+			(xy 175.26 118.11) (xy 175.26 121.92)
 		)
 		(stroke
@@
 	(wire
 		(pts
-			(xy 146.05 105.41) (xy 173.99 105.41)
+			(xy 146.05 105.41) (xy 175.26 105.41)
 		)
 		(stroke
@@
 	)
 	(hierarchical_label "RESET"
-		(shape input)
+		(shape output)
 		(at 146.05 90.17 0)
 		(effects
@@
 	)
 	(hierarchical_label "READY"
-		(shape input)
+		(shape output)
 		(at 146.05 85.09 0)
 		(effects
@@
 	)
 	(hierarchical_label "CLK"
-		(shape input)
+		(shape output)
 		(at 146.05 80.01 0)
 		(effects
@@
 	)
 	(hierarchical_label "RESET"
-		(shape input)
+		(shape output)
 		(at 207.01 100.33 90)
 		(effects
@@
 	(symbol
 		(lib_id "power:GND")
-		(at 173.99 129.54 0)
+		(at 175.26 129.54 0)
 		(unit 1)
 		(body_style 1)
@@
 		(fields_autoplaced yes)
 		(property "Reference" "#PWR02"
-			(at 173.99 135.89 0)
+			(at 175.26 135.89 0)
 			(hide yes)
 			(show_name no)
@@
 		)
 		(property "Value" "GND"
-			(at 173.99 134.62 0)
+			(at 175.26 134.62 0)
 			(show_name no)
 			(do_not_autoplace no)
@@
 		)
 		(property "Footprint" ""
-			(at 173.99 129.54 0)
+			(at 175.26 129.54 0)
 			(hide yes)
 			(show_name no)
@@
 		)
 		(property "Datasheet" ""
-			(at 173.99 129.54 0)
+			(at 175.26 129.54 0)
 			(hide yes)
 			(show_name no)
@@
 		)
 		(property "Description" "Power symbol creates a global label with name \"GND\" , ground"
-			(at 173.99 129.54 0)
+			(at 175.26 129.54 0)
 			(hide yes)
 			(show_name no)
@@
 	(symbol
 		(lib_id "Device:C")
-		(at 173.99 125.73 0)
+		(at 175.26 125.73 0)
 		(unit 1)
 		(body_style 1)
@@
 		(fields_autoplaced yes)
 		(property "Reference" "C2"
-			(at 177.8 124.4599 0)
+			(at 179.07 124.4599 0)
 			(show_name no)
 			(do_not_autoplace no)
@@
 		)
 		(property "Value" "33 pF"
-			(at 177.8 126.9999 0)
+			(at 179.07 126.9999 0)
 			(show_name no)
 			(do_not_autoplace no)
@@
 		)
 		(property "Footprint" "Capacitor_THT:C_Disc_D5.0mm_W2.5mm_P5.00mm"
-			(at 174.9552 129.54 0)
+			(at 176.2252 129.54 0)
 			(hide yes)
 			(show_name no)
@@
 		)
 		(property "Datasheet" ""
-			(at 173.99 125.73 0)
+			(at 175.26 125.73 0)
 			(hide yes)
 			(show_name no)
@@
 		)
 		(property "Description" "Unpolarized capacitor"
-			(at 173.99 125.73 0)
+			(at 175.26 125.73 0)
 			(hide yes)
 			(show_name no)
@@
 	(symbol
 		(lib_id "Device:Crystal")
-		(at 165.1 118.11 0)
+		(at 166.37 118.11 0)
 		(unit 1)
 		(body_style 1)
@@
 		(fields_autoplaced yes)
 		(property "Reference" "Y1"
-			(at 165.1 110.49 0)
+			(at 166.37 110.49 0)
 			(show_name no)
 			(do_not_autoplace no)
@@
 		)
 		(property "Value" "14.31818 MHz"
-			(at 165.1 113.03 0)
+			(at 166.37 113.03 0)
 			(show_name no)
 			(do_not_autoplace no)
@@
 		)
 		(property "Footprint" "Crystal:Crystal_HC49-U_Vertical"
-			(at 165.1 118.11 0)
+			(at 166.37 118.11 0)
 			(hide yes)
 			(show_name no)
@@
 		)
 		(property "Datasheet" ""
-			(at 165.1 118.11 0)
+			(at 166.37 118.11 0)
 			(hide yes)
 			(show_name no)
@@
 		)
 		(property "Description" "Two pin crystal"
-			(at 165.1 118.11 0)
-			(hide yes)
-			(show_name no)
+			(at 166.37 118.11 0)
+			(hide yes)
+			(show_name no)

Commit message: Update 8086-mainboard scheme
Parts:
- added JP1: Jumper_2_Open, Connector_PinHeader_2.54mm:PinHeader_1x02_P2.54mm_Vertical, symbol Jumper:Jumper_2_Open
Connections:
- net GND: now also JP1.2 (B)
- net at R2.2, U2.4 (RDY1), U2.6 (RDY2): now also JP1.1 (A)

Commit message: Finalize 8088 mainboard rev1.0 for production
Parts:
- removed JP1: Jumper_2_Open, Connector_PinHeader_2.54mm:PinHeader_1x02_P2.54mm_Vertical, symbol Jumper:Jumper_2_Open
- added D3, D4: BAT85, Diode_THT:D_DO-35_SOD27_P7.62mm_Horizontal, symbol Diode:BAT85
- added J5: Ext CLK, Connector_PinHeader_2.54mm:PinHeader_1x02_P2.54mm_Vertical, symbol Connector_Generic:Conn_01x02
- added R6: 1k, Resistor_THT:R_Axial_DIN0207_L6.3mm_D2.5mm_P7.62mm_Horizontal, symbol Device:R
- added R8, R9: 10k, Resistor_THT:R_Axial_DIN0207_L6.3mm_D2.5mm_P7.62mm_Horizontal, symbol Device:R
- added SW2: SW_DIP_x02, Button_Switch_THT:SW_DIP_SPSTx02_Slide_9.78x7.26mm_W7.62mm_P2.54mm, symbol Switch:SW_DIP_x02
- C5: renamed from C4; footprint Capacitor_THT:CP_Radial_D5.0mm_P2.00mm -> Capacitor_THT:CP_Radial_D4.0mm_P1.50mm
- R3: renamed from R4; value 330 -> 680
- U5: renamed from U2; footprint Package_DIP:DIP-18_W7.62mm -> Package_DIP:DIP-18_W7.62mm_Socket
- renumbered C3 to C6, C1 to C7, C2 to C8
Connections:
- net GND: now also U5.1 (CSYNC), D4.2 (A), J5.2 (Pin_2), R8.2, R9.2, SW2.1; no longer U5.13 (F/~{C}), U5.14 (EFI)
- net VCC: now also D3.1 (K), SW2.2
- net RDY: now reaches R2.2, U5.4 (RDY1), U5.6 (RDY2)
- net RDY: now also SW2.4
- new net: D3.2 (A), D4.1 (K), R6.1, R9.1, U5.14 (EFI)
- new net: R8.1, SW2.3, U5.13 (F/~{C})
- new net: J5.1 (Pin_1), R6.2
- no-connect marks 3 -> 2
Other:
- moved on the sheet: C5, C6, C7, C8, D2, R1, R2, R3, SW1, U5, Y1

Commit message: Add LCD module and demo BIOS
Parts:
- removed C7, C8: 33 pF, Capacitor_THT:C_Disc_D5.0mm_W2.5mm_P5.00mm, symbol Device:C
