File: hardware/kicad/IO_DECODER.kicad_sch (KiCad schematic)
At the start: 2 parts, among them U7 74LS138

Commit message: Add mainboard v2.0
Parts:
- C8: renamed from C10; footprint Capacitor_THT:C_Disc_D5.0mm_W2.5mm_P5.00mm -> Capacitor_SMD:C_0805_2012Metric
Connections:
- net EXP_IO_CS4: now reaches U7.11 (O4)
- net IO_PIT_CS: now reaches U7.13 (O2)
- net IO_PIC_CS: now reaches U7.14 (O1)
- net IO_UART_CS: now reaches U7.7 (O7)
- net IO_EXP0_CS renamed EXP_IO_CS5
- net IO_EXP1_CS renamed EXP_IO_CS6
- no-connect marks 6 -> 2
Changed lines of the file:
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@@
 	)
 	(no_connect
-		(at 151.13 83.82)
+		(at 151.13 78.74)
 	)
 	(no_connect
 		(at 151.13 86.36)
 	)
-	(no_connect
-		(at 151.13 78.74)
-	)
-	(no_connect
-		(at 151.13 81.28)
-	)
-	(no_connect
-		(at 151.13 88.9)
-	)
-	(no_connect
-		(at 151.13 96.52)
-	)
 	(wire
 		(pts
@@
 			(width 0)
 			(type default)
+		)
+	)
+	(hierarchical_label "EXP_IO_CS4"
+		(shape output)
+		(at 151.13 88.9 0)
+		(effects
+			(font
+				(size 1.27 1.27)
+			)
+			(justify left)
+		)
+	)
+	(hierarchical_label "IO_PIT_CS"
+		(shape output)
+		(at 151.13 83.82 0)
+		(effects
+			(font
+				(size 1.27 1.27)
+			)
+			(justify left)
 		)
 	)
@@
 		)
 	)
+	(hierarchical_label "IO_UART_CS"
+		(shape output)
+		(at 151.13 96.52 0)
+		(effects
+			(font
+				(size 1.27 1.27)
+			)
+			(justify left)
+		)
+	)
 	(hierarchical_label "A6"
 		(shape input)
@@
 		)
 	)
-	(hierarchical_label "IO_EXP1_CS"
+	(hierarchical_label "EXP_IO_CS6"
 		(shape output)
 		(at 151.13 93.98 0)
@@
 		)
 	)
-	(hierarchical_label "IO_EXP0_CS"
+	(hierarchical_label "EXP_IO_CS5"
 		(shape output)
 		(at 151.13 91.44 0)
+		(effects
+			(font
+				(size 1.27 1.27)
+			)
+			(justify left)
+		)
+	)
+	(hierarchical_label "IO_PIC_CS"
+		(shape output)
+		(at 151.13 81.28 0)
 		(effects
 			(font
@@
 		(dnp no)
 		(fields_autoplaced yes)
-		(property "Reference" "#PWR040"
+		(property "Reference" "#PWR041"
 			(at 106.68 67.31 0)
 			(hide yes)
@@
 			(project "8088-mainboard"
 				(path "/15ce4f45-6f32-456e-874c-aac11293789a/c64b3a1d-9cdf-4d26-8a62-60cbadd711b0"
-					(reference "#PWR040")
+					(reference "#PWR041")
 					(unit 1)
 				)
@@
 		(in_pos_files yes)
 		(dnp no)
-		(property "Reference" "#PWR041"
+		(property "Reference" "#PWR042"
 			(at 124.46 66.04 0)
 			(hide yes)
@@
 			(project "8088-mainboard"
 				(path "/15ce4f45-6f32-456e-874c-aac11293789a/c64b3a1d-9cdf-4d26-8a62-60cbadd711b0"
-					(reference "#PWR041")
+					(reference "#PWR042")
 					(unit 1)
 				)
@@
 		(dnp no)
 		(fields_autoplaced yes)
-		(property "Reference" "#PWR042"
+		(property "Reference" "#PWR043"
 			(at 124.46 110.49 0)
 			(hide yes)
@@
 			(project "8088-mainboard"
 				(path "/15ce4f45-6f32-456e-874c-aac11293789a/c64b3a1d-9cdf-4d26-8a62-60cbadd711b0"
-					(reference "#PWR042")
+					(reference "#PWR043")
 					(unit 1)
 				)
@@
 		(dnp no)
 		(fields_autoplaced yes)
-		(property "Reference" "#PWR039"
+		(property "Reference" "#PWR040"
 			(at 105.41 96.52 0)
 			(hide yes)
@@
 			(project "8088-mainboard"
 				(path "/15ce4f45-6f32-456e-874c-aac11293789a/c64b3a1d-9cdf-4d26-8a62-60cbadd711b0"
-					(reference "#PWR039")
+					(reference "#PWR040")
 					(unit 1)
 				)
@@
 		(in_pos_files yes)
 		(dnp no)
-		(property "Reference" "C10"
+		(property "Reference" "C8"
 			(at 116.84 61.214 0)
 			(show_name no)
@@
 			)
 		)
-		(property "Footprint" "Capacitor_THT:C_Disc_D5.0mm_W2.5mm_P5.00mm"
+		(property "Footprint" "Capacitor_SMD:C_0805_2012Metric"
 			(at 113.03 68.2752 0)
 			(hide yes)
@@
 			(project "8088-mainboard"
 				(path "/15ce4f45-6f32-456e-874c-aac11293789a/c64b3a1d-9cdf-4d26-8a62-60cbadd711b0"
-					(reference "C10")
+					(reference "C8")
 					(unit 1)
 				)
@@
 		(dnp no)
 		(fields_autoplaced yes)
-		(property "Reference" "#PWR038"
+		(property "Reference" "#PWR039"
 			(at 105.41 93.98 0)
 			(hide yes)
@@
 			(project "8088-mainboard"
 				(path "/15ce4f45-6f32-456e-874c-aac11293789a/c64b3a1d-9cdf-4d26-8a62-60cbadd711b0"
-					(reference "#PWR038")
+					(reference "#PWR039")
 					(unit 1)
 				)
