File: hardware/kicad/RAM.kicad_sch (KiCad schematic)
At the start: 2 parts, among them U9 HM62256BLP

Commit message: Add mainboard v2.0
Parts:
- removed U9: HM62256BLP, Package_DIP:DIP-28_W15.24mm_Socket, symbol Memory_RAM:HM62256BLP
- added C10, C11, C13, C14: 100nF, Capacitor_SMD:C_0805_2012Metric, symbol Device:C
- added U10, U11, U12, U13, U9: AS6C1008-55PCN, Package_DIP:DIP-32_W15.24mm_Socket, symbol Memory_RAM:AS6C1008-xxP
- C12: footprint Capacitor_THT:C_Disc_D5.0mm_W2.5mm_P5.00mm -> Capacitor_SMD:C_0805_2012Metric
Connections:
- net A0: now also U10.12 (A0), U11.12 (A0), U12.12 (A0), U13.12 (A0), U9.12 (A0)
- net A1: now also U10.11 (A1), U11.11 (A1), U12.11 (A1), U13.11 (A1), U9.11 (A1)
- net A10: now also U10.23 (A10), U11.23 (A10), U12.23 (A10), U13.23 (A10), U9.23 (A10)
- net A11: now also U10.25 (A11), U11.25 (A11), U12.25 (A11), U13.25 (A11), U9.25 (A11)
- net A12: now also U10.4 (A12), U11.4 (A12), U12.4 (A12), U13.4 (A12), U9.4 (A12)
- net A13: now also U10.28 (A13), U11.28 (A13), U12.28 (A13), U13.28 (A13), U9.28 (A13)
- net A14: now also U10.3 (A14), U11.3 (A14), U12.3 (A14), U13.3 (A14), U9.3 (A14)
- net A2: now also U10.10 (A2), U11.10 (A2), U12.10 (A2), U13.10 (A2), U9.10 (A2)
- net A3: now also U10.9 (A3), U11.9 (A3), U12.9 (A3), U13.9 (A3), U9.9 (A3)
- net A4: now also U10.8 (A4), U11.8 (A4), U12.8 (A4), U13.8 (A4), U9.8 (A4)
- net A5: now also U10.7 (A5), U11.7 (A5), U12.7 (A5), U13.7 (A5), U9.7 (A5)
- net A6: now also U10.6 (A6), U11.6 (A6), U12.6 (A6), U13.6 (A6), U9.6 (A6)
- net A7: now also U10.5 (A7), U11.5 (A7), U12.5 (A7), U13.5 (A7), U9.5 (A7)
- net A8: now also U10.27 (A8), U11.27 (A8), U12.27 (A8), U13.27 (A8), U9.27 (A8)
- net A9: now also U10.26 (A9), U11.26 (A9), U12.26 (A9), U13.26 (A9), U9.26 (A9)
- net D0: now also U10.13 (DQ0), U11.13 (DQ0), U12.13 (DQ0), U13.13 (DQ0), U9.13 (DQ0)
- net D1: now also U10.14 (DQ1), U11.14 (DQ1), U12.14 (DQ1), U13.14 (DQ1), U9.14 (DQ1)
- net D2: now also U10.15 (DQ2), U11.15 (DQ2), U12.15 (DQ2), U13.15 (DQ2), U9.15 (DQ2)
- net D3: now also U10.17 (DQ3), U11.17 (DQ3), U12.17 (DQ3), U13.17 (DQ3), U9.17 (DQ3)
- net D4: now also U10.18 (DQ4), U11.18 (DQ4), U12.18 (DQ4), U13.18 (DQ4), U9.18 (DQ4)
- net D5: now also U10.19 (DQ5), U11.19 (DQ5), U12.19 (DQ5), U13.19 (DQ5), U9.19 (DQ5)
- net D6: now also U10.20 (DQ6), U11.20 (DQ6), U12.20 (DQ6), U13.20 (DQ6), U9.20 (DQ6)
- net D7: now also U10.21 (DQ7), U11.21 (DQ7), U12.21 (DQ7), U13.21 (DQ7), U9.21 (DQ7)
- net GND: now also C10.2, C11.2, C13.2, C14.2, U10.16 (GND), U11.16 (GND), U12.16 (GND), U13.16 (GND), U9.16 (GND)
- net RAM_BANK0_CS: now also U9.22 (~{CS1}/~{CE1})
- net RD: now also U10.24 (~{OE}), U11.24 (~{OE}), U12.24 (~{OE}), U13.24 (~{OE}), U9.24 (~{OE})
- net VCC: now also C10.1, C11.1, C13.1, C14.1, U10.30 (CS2/CE2), U10.32 (VCC), U11.30 (CS2/CE2), U11.32 (VCC), U12.30 (CS2/CE2), U12.32 (VCC), U13.30 (CS2/CE2), U13.32 (VCC), U9.30 (CS2/CE2), U9.32 (VCC)
- net WR: now also U10.29 (~{WE}), U11.29 (~{WE}), U12.29 (~{WE}), U13.29 (~{WE}), U9.29 (~{WE})
- new net A15: U10.31 (A15), U11.31 (A15), U12.31 (A15), U13.31 (A15), U9.31 (A15)
- new net A16: U10.2 (A16), U11.2 (A16), U12.2 (A16), U13.2 (A16), U9.2 (A16)
- new net RAM_BANK1_CS: U10.22 (~{CS1}/~{CE1})
- new net RAM_BANK2_CS: U11.22 (~{CS1}/~{CE1})
- new net RAM_BANK3_CS: U12.22 (~{CS1}/~{CE1})
- new net RAM_BANK4_CS: U13.22 (~{CS1}/~{CE1})
