File: hardware/kicad/uart.kicad_sch (KiCad schematic)
At the start: 14 parts, among them J2 Ext Res, J3 Ext CLK, SW2 Reset, U5 8284, Y1 14.31818 MHz

Commit message: Add mainboard v2.0
Parts:
- removed C5: 10 uF, Capacitor_THT:CP_Radial_D4.0mm_P1.50mm, symbol Device:C
- removed C6: 100 nF, Capacitor_SMD:C_0805_2012Metric, symbol Device:C
- removed D1: RST LED, LED_SMD:LED_0805_2012Metric, symbol Device:LED
- removed J2: Ext Res, Connector_PinHeader_2.54mm:PinHeader_1x02_P2.54mm_Vertical, symbol Connector_Generic:Conn_01x02
- removed J3: Ext CLK, Connector_PinHeader_2.54mm:PinHeader_1x02_P2.54mm_Vertical, symbol Connector_Generic:Conn_01x02
- removed R4: 680, Resistor_SMD:R_0805_2012Metric, symbol Device:R
- removed R5, R6, R7, R9: 10k, Resistor_SMD:R_0805_2012Metric, symbol Device:R
- removed R8: 1k, Resistor_SMD:R_0805_2012Metric, symbol Device:R
- removed SW2: Reset, Button_Switch_THT:SW_PUSH_6mm, symbol Switch:SW_Push
- removed U5: 8284, Package_DIP:DIP-18_W7.62mm_Socket, symbol Timer:8284
- removed Y1: 14.31818 MHz, Crystal:Crystal_HC49-U_Vertical, symbol Device:Crystal
- added C16: 22pF, Capacitor_SMD:C_0805_2012Metric, symbol Device:C
- added C17: 47pF, Capacitor_SMD:C_0805_2012Metric, symbol Device:C
- added C18: 100nF, Capacitor_SMD:C_0805_2012Metric, symbol Device:C
- added J9: CP2102 Module, Connector_PinHeader_2.54mm:PinHeader_1x03_P2.54mm_Vertical, symbol Connector_Generic:Conn_01x03
- added R13: 1M, Resistor_SMD:R_0805_2012Metric, symbol Device:R
- added R14: 1.5k, Resistor_SMD:R_0805_2012Metric, symbol Device:R
- added R15, R16, R17, R18: 10k, Resistor_SMD:R_0805_2012Metric, symbol Device:R
- added R19: 1k, Resistor_SMD:R_0805_2012Metric, symbol Device:R
- added R20: 2K, Resistor_SMD:R_0805_2012Metric, symbol Device:R
- added U14: GM16C550, Package_DIP:DIP-40_W15.24mm_Socket, symbol Interface_UART:16550
- added Y2: 1.8432 MHz, Crystal:Crystal_HC49-U_Vertical, symbol Device:Crystal
Connections:
- net GND: now also C16.1, C17.1, C18.2, J9.1 (Pin_1), R20.1, U14.19 (WR), U14.20 (GND), U14.22 (RD)
- net RESET: now also U14.35 (MR)
- net VCC: now also C18.1, R15.1, R16.1, R17.1, R18.1, U14.12 (CS0), U14.13 (CS1), U14.40 (VCC)
- new net: C17.2, R13.1, R14.1, Y2.1
- new net: C16.2, R13.2, U14.16 (XIN), Y2.2
- new net: R15.2, U14.39 (~{RI})
- new net: R18.2, U14.36 (~{CTS})
- new net: R19.1, U14.11 (SOUT)
- new net: U14.15 (~{BAUDOUT}), U14.9 (RCLK)
- new net: R14.2, U14.17 (XOUT)
- new net: R17.2, U14.37 (~{DSR})
- new net: R16.2, U14.38 (~{DCD})
- new net A0: U14.28 (A0)
- new net A1: U14.27 (A1)
- new net A2: U14.26 (A2)
- new net ALE: U14.25 (~{ADS})
- new net D0: U14.1 (D0)
- new net D1: U14.2 (D1)
- new net D2: U14.3 (D2)
- new net D3: U14.4 (D3)
- new net D4: U14.5 (D4)
- new net D5: U14.6 (D5)
- new net D6: U14.7 (D6)
- new net D7: U14.8 (D7)
- new net IO_UART_CS: U14.14 (~{CS2})
- new net RD: U14.21 (~{RD})
- new net RXI: J9.3 (Pin_3), R19.2, R20.2
- new net TXD: J9.2 (Pin_2), U14.10 (SIN)
- new net UART_IRQ: U14.30 (INTR)
- new net WR: U14.18 (~{WR})
- no-connect marks 1 -> 7
