File: hardware/kicad/EXPANSION_CONNECTOR.kicad_sch (KiCad schematic)
At the start: 2 parts, among them J2 Exp0, J3 Exp1

Commit message: Add mainboard v2.0
Parts:
- removed J2: Exp0, Connector_IDC:IDC-Header_2x20_P2.54mm_Vertical, symbol Connector_Generic:Conn_02x20_Odd_Even
- removed J3: Exp1, Connector_IDC:IDC-Header_2x20_P2.54mm_Vertical, symbol Connector_Generic:Conn_02x20_Odd_Even
- added J4: EXP_0_A, Connector_PinSocket_2.54mm:PinSocket_2x20_P2.54mm_Vertical, symbol Connector_Generic:Conn_02x20_Counter_Clockwise
- added J5: EXP_0_B, Connector_PinSocket_2.54mm:PinSocket_2x10_P2.54mm_Vertical, symbol Connector_Generic:Conn_02x10_Counter_Clockwise
- added J6: EXP_1_A, Connector_PinSocket_2.54mm:PinSocket_2x20_P2.54mm_Vertical, symbol Connector_Generic:Conn_02x20_Counter_Clockwise
- added J7: EXP_1_B, Connector_PinSocket_2.54mm:PinSocket_2x10_P2.54mm_Vertical, symbol Connector_Generic:Conn_02x10_Counter_Clockwise
Connections:
- net A0: now also J4.40 (Pin_40), J6.40 (Pin_40)
- net A1: now also J4.39 (Pin_39), J6.39 (Pin_39)
- net A10: now also J4.30 (Pin_30), J6.30 (Pin_30)
- net A11: now also J4.29 (Pin_29), J6.29 (Pin_29)
- net A12: now also J4.28 (Pin_28), J6.28 (Pin_28)
- net A13: now also J4.27 (Pin_27), J6.27 (Pin_27)
- net A14: now also J4.26 (Pin_26), J6.26 (Pin_26)
- net A15: now also J4.25 (Pin_25), J6.25 (Pin_25)
- net A16: now also J4.24 (Pin_24), J6.24 (Pin_24)
- net A17: now also J4.23 (Pin_23), J6.23 (Pin_23)
- net A18: now also J4.22 (Pin_22), J6.22 (Pin_22)
- net A19: now also J4.21 (Pin_21), J6.21 (Pin_21)
- net A2: now also J4.38 (Pin_38), J6.38 (Pin_38)
- net A3: now also J4.37 (Pin_37), J6.37 (Pin_37)
- net A4: now also J4.36 (Pin_36), J6.36 (Pin_36)
- net A5: now also J4.35 (Pin_35), J6.35 (Pin_35)
- net A6: now also J4.34 (Pin_34), J6.34 (Pin_34)
- net A7: now also J4.33 (Pin_33), J6.33 (Pin_33)
- net A8: now also J4.32 (Pin_32), J6.32 (Pin_32)
- net A9: now also J4.31 (Pin_31), J6.31 (Pin_31)
- net ALE: now also J4.9 (Pin_9), J6.9 (Pin_9)
- net CLK: now also J5.2 (Pin_2), J7.2 (Pin_2)
- net D0: now also J4.18 (Pin_18), J6.18 (Pin_18)
- net D1: now also J4.17 (Pin_17), J6.17 (Pin_17)
- net D2: now also J4.16 (Pin_16), J6.16 (Pin_16)
- net D3: now also J4.15 (Pin_15), J6.15 (Pin_15)
- net D4: now also J4.14 (Pin_14), J6.14 (Pin_14)
- net D5: now also J4.13 (Pin_13), J6.13 (Pin_13)
- net D6: now also J4.12 (Pin_12), J6.12 (Pin_12)
- net D7: now also J4.11 (Pin_11), J6.11 (Pin_11)
- net GND: now also J4.1 (Pin_1), J4.10 (Pin_10), J4.19 (Pin_19), J4.20 (Pin_20), J5.1 (Pin_1), J5.10 (Pin_10), J5.19 (Pin_19), J5.20 (Pin_20), J6.1 (Pin_1), J6.10 (Pin_10), J6.19 (Pin_19), J6.20 (Pin_20), J7.1 (Pin_1), J7.10 (Pin_10), J7.19 (Pin_19), J7.20 (Pin_20)
- net IOM: now also J4.3 (Pin_3), J6.3 (Pin_3)
- net RD: now also J4.5 (Pin_5), J6.5 (Pin_5)
- net RDY: now also J4.6 (Pin_6), J6.6 (Pin_6)
- net RESET: now also J4.7 (Pin_7), J6.7 (Pin_7)
- net VCC: now also J4.2 (Pin_2), J6.2 (Pin_2)
- net WR: now also J4.4 (Pin_4), J6.4 (Pin_4)
- new net DEN: J5.6 (Pin_6), J7.6 (Pin_6)
- new net DT_R: J5.5 (Pin_5), J7.5 (Pin_5)
- new net EXP_IO_CS4: J5.7 (Pin_7), J7.7 (Pin_7)
- new net EXP_IO_CS5: J5.8 (Pin_8), J7.8 (Pin_8)
- new net EXP_IO_CS6: J5.9 (Pin_9), J7.9 (Pin_9)
- new net EXP_IRQ1: J5.13 (Pin_13), J7.13 (Pin_13)
- new net EXP_IRQ2: J5.14 (Pin_14), J7.14 (Pin_14)
- new net EXP_IRQ3: J5.15 (Pin_15), J7.15 (Pin_15)
- new net EXP_IRQ5: J5.16 (Pin_16), J7.16 (Pin_16)
- new net EXP_IRQ6: J5.17 (Pin_17), J7.17 (Pin_17)
- new net EXP_IRQ7: J5.18 (Pin_18), J7.18 (Pin_18)
- new net EXP_MEM_CS5: J5.11 (Pin_11), J7.11 (Pin_11)
- new net EXP_MEM_CS6: J5.12 (Pin_12), J7.12 (Pin_12)
- new net HLDA: J5.4 (Pin_4), J7.4 (Pin_4)
- new net HOLD: J5.3 (Pin_3), J7.3 (Pin_3)
- new net NMI: J4.8 (Pin_8), J6.8 (Pin_8)

Commit message: Update mainboard and expansion modules
Parts:
- added R29, R30, R31, R32, R33, R34, R35, R36, R37, R38, R39, R40, R41, R42, R43, R44: 33, Resistor_SMD:R_0805_2012Metric, symbol Device:R
Connections:
- net D0: now also R36.2, R44.2; no longer J4.18 (Pin_18), J6.18 (Pin_18)
- net D1: now also R35.2, R43.2; no longer J4.17 (Pin_17), J6.17 (Pin_17)
- net D2: now also R34.2, R42.2; no longer J4.16 (Pin_16), J6.16 (Pin_16)
- net D3: now also R33.2, R41.2; no longer J4.15 (Pin_15), J6.15 (Pin_15)
- net D4: now also R32.2, R40.2; no longer J4.14 (Pin_14), J6.14 (Pin_14)
- net D5: now also R31.2, R39.2; no longer J4.13 (Pin_13), J6.13 (Pin_13)
- net D6: now also R30.2, R38.2; no longer J4.12 (Pin_12), J6.12 (Pin_12)
- net D7: now also R29.2, R37.2; no longer J4.11 (Pin_11), J6.11 (Pin_11)
- new net: J4.11 (Pin_11), R29.1
- new net: J6.12 (Pin_12), R38.1
- new net: J6.16 (Pin_16), R42.1
- new net: J4.16 (Pin_16), R34.1
- new net: J4.18 (Pin_18), R36.1
- new net: J4.15 (Pin_15), R33.1
- new net: J4.17 (Pin_17), R35.1
- new net: J6.11 (Pin_11), R37.1
- new net: J6.14 (Pin_14), R40.1
- new net: J4.13 (Pin_13), R31.1
- new net: J6.15 (Pin_15), R41.1
- new net: J6.13 (Pin_13), R39.1
- new net: J6.17 (Pin_17), R43.1
- new net: J6.18 (Pin_18), R44.1
- new net: J4.14 (Pin_14), R32.1
- new net: J4.12 (Pin_12), R30.1
Other:
- moved on the sheet: J5, J6, J7
