File: hardware/kicad/8088-mainboard.kicad_pcb (KiCad board)
At the start: 2 copper layers, 185.4 x 160 mm, 104 parts, among them J1 Conn_01x10, J10 Conn_01x04, J11 Conn_01x04, J2 Ext Res, J3 Ext CLK, J4 EXP_0_A, J5 EXP_0_B, J6 EXP_1_A, J7 EXP_1_B, J8 POWER 5v, J9 CP2102 Module, Q1 NDP6020P, SW1 SW_DIP_x03, SW2 Reset, U1 8088_Min_Mode, U10 AS6C1008-55PCN, U11 AS6C1008-55PCN, U12 AS6C1008-55PCN, U13 AS6C1008-55PCN, U14 GM16C550, U15 8259A-2, U16 8254, U17 74LS74, U2 74LS373, U3 74LS373, U4 74LS245, U5 8284, U6 74LS138, U7 74LS138, U8 28C256, U9 AS6C1008-55PCN, Y1 14.31818 MHz, Y2 1.8432 MHz

Commit message: Update schema
Connections:
- net /IO_DECODER/IO_PIC_CS renamed /IO_PIC_CS
- net /IO_DECODER/IO_UART_CS renamed /IO_UART_CS
