File: hardware/kicad/8088-mainboard.kicad_sch (KiCad schematic)
At the start: 0 parts

Commit message: Add mainboard v2.0
Parts:
- added SW1: SW_DIP_x03, Button_Switch_THT:SW_DIP_SPSTx03_Slide_9.78x9.8mm_W7.62mm_P2.54mm, symbol Switch:SW_DIP_x03
Connections:
- net RDY: now also SW1.6
- net WR: now also SW1.2
- new net CLOCK_EFI_SW: SW1.4
- new net GND: SW1.1
- new net ROM_WE_SW: SW1.5
- new net VCC: SW1.3
Other:
- added sheet PIC (PIC.kicad_sch)
- added sheet PIT (PIT.kicad_sch)
- added sheet UART (uart.kicad_sch)
- sheet CLOCK ports: added EFI_SW, PCLK; removed none
- sheet CPU ports: added DEN, DT_R, HLDA, HOLD, INTA, INTR, NMI; removed none
- sheet EXPANSION_CONNECTOR ports: added DEN, DT_R, EXP_IO_CS4, EXP_IO_CS5, EXP_IO_CS6, EXP_IRQ1, EXP_IRQ2, EXP_IRQ3, EXP_IRQ5, EXP_IRQ6, EXP_IRQ7, EXP_MEM_CS5, EXP_MEM_CS6, HLDA, HOLD, NMI; removed IO_EXP0_CS, IO_EXP1_CS, MEM_EXP0_CS, MEM_EXP1_CS
- sheet IO_DECODER ports: added EXP_IO_CS4, EXP_IO_CS5, EXP_IO_CS6, IO_PIC_CS, IO_PIT_CS, IO_UART_CS; removed IO_EXP0_CS, IO_EXP1_CS
- sheet MEM_DECODER ports: added EXP_MEM_CS5, EXP_MEM_CS6, RAM_BANK1_CS, RAM_BANK2_CS, RAM_BANK3_CS, RAM_BANK4_CS; removed MEM_EXP0_CS, MEM_EXP1_CS
- sheet RAM ports: added RAM_BANK1_CS, RAM_BANK2_CS, RAM_BANK3_CS, RAM_BANK4_CS; removed none
- sheet ROM ports: added WE_SW; removed none

Commit message: Update schema
Other:
- moved on the sheet: SW1
