File: hardware/kicad/CLOCK.kicad_sch (KiCad schematic)
At the start: 16 parts, among them J5 Ext CLK, SW1 Reset, SW2 SW_DIP_x02, U5 8284, Y1 14.31818 MHz

Commit message: Add mainboard v2.0 (#6)
* Add mainboard v2.0
Parts:
- removed D3, D4: BAT85, Diode_THT:D_DO-35_SOD27_P7.62mm_Horizontal, symbol Diode:BAT85
- removed SW2: SW_DIP_x02, Button_Switch_THT:SW_DIP_SPSTx02_Slide_9.78x7.26mm_W7.62mm_P2.54mm, symbol Switch:SW_DIP_x02
- added J2: Ext Res, Connector_PinHeader_2.54mm:PinHeader_1x02_P2.54mm_Vertical, symbol Connector_Generic:Conn_01x02
- C6: footprint Capacitor_THT:C_Disc_D5.0mm_W2.5mm_P5.00mm -> Capacitor_SMD:C_0805_2012Metric
- D1: renamed from D2; footprint LED_THT:LED_D3.0mm -> LED_SMD:LED_0805_2012Metric
- R4: renamed from R3; footprint Resistor_THT:R_Axial_DIN0207_L6.3mm_D2.5mm_P7.62mm_Horizontal -> Resistor_SMD:R_0805_2012Metric
- R5: renamed from R1; footprint Resistor_THT:R_Axial_DIN0207_L6.3mm_D2.5mm_P7.62mm_Horizontal -> Resistor_SMD:R_0805_2012Metric
- R6: renamed from R2; footprint Resistor_THT:R_Axial_DIN0207_L6.3mm_D2.5mm_P7.62mm_Horizontal -> Resistor_SMD:R_0805_2012Metric
- R7: renamed from R8; footprint Resistor_THT:R_Axial_DIN0207_L6.3mm_D2.5mm_P7.62mm_Horizontal -> Resistor_SMD:R_0805_2012Metric
- R8: renamed from R6; footprint Resistor_THT:R_Axial_DIN0207_L6.3mm_D2.5mm_P7.62mm_Horizontal -> Resistor_SMD:R_0805_2012Metric
- R9: footprint Resistor_THT:R_Axial_DIN0207_L6.3mm_D2.5mm_P7.62mm_Horizontal -> Resistor_SMD:R_0805_2012Metric
- renumbered J5 to J3, SW1 to SW2
Connections:
- net GND: now also J3.1 (Pin_1), J2.1 (Pin_1); no longer J3.2 (Pin_2)
- net RES: now also J2.2 (Pin_2)
- net EFI_SW: now reaches R7.1, U5.13 (F/~{C})
- net PCLK: now reaches U5.2 (PCLK)
- net at R8.2: now also J3.2 (Pin_2); no longer J3.1 (Pin_1)
- no-connect marks 2 -> 1
Other:
- moved on the sheet: C5, C6, D1, J3, R4, R5, R6, R7, R8, R9, SW2, U5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
