File: hardware/kicad/CPU.kicad_sch (KiCad schematic)
At the start: 9 parts, among them J1 Conn_01x10, U1 8088_Min_Mode, U2 74LS373, U3 74LS373, U4 74LS245

Commit message: Add mainboard v2.0
Parts:
- added R1, R2, R3: 10k, Resistor_SMD:R_0805_2012Metric, symbol Device:R
- C1, C2, C3, C4: footprint Capacitor_THT:C_Disc_D5.0mm_W2.5mm_P5.00mm -> Capacitor_SMD:C_0805_2012Metric
Connections:
- net ALE: now also J1.10 (Pin_10); no longer J1.5 (Pin_5)
- net DEN: now also J1.5 (Pin_5); no longer J1.10 (Pin_10)
- net GND: now also R1.2, R2.2, R3.2; no longer U1.17 (NMI), U1.18 (INTR), U1.31 (HOLD)
- net INTA: now reaches U1.24 (~{INTA})
- net HLDA: now reaches U1.30 (HLDA)
- new net HOLD: R1.1, U1.31 (HOLD)
- new net INTR: R2.1, U1.18 (INTR)
- new net NMI: R3.1, U1.17 (NMI)
- no-connect marks 7 -> 5
Other:
- moved on the sheet: C1, U1

Commit message: Update schema
Other:
- moved on the sheet: C1, C2, C3, C4, R1, R2, R3, U1, U2, U3, U4
