File: hardware/kicad/MEM_DECODER.kicad_sch (KiCad schematic)
At the start: 2 parts, among them U6 74LS138

Commit message: Add mainboard v2.0
Parts:
- C7: renamed from C9; footprint Capacitor_THT:C_Disc_D5.0mm_W2.5mm_P5.00mm -> Capacitor_SMD:C_0805_2012Metric
Connections:
- net RAM_BANK3_CS: now reaches U6.12 (O3)
- net RAM_BANK2_CS: now reaches U6.13 (O2)
- net RAM_BANK1_CS: now reaches U6.14 (O1)
- net EXP_MEM_CS6: now reaches U6.9 (O6)
- net MEM_EXP0_CS renamed RAM_BANK4_CS
- net MEM_EXP1_CS renamed EXP_MEM_CS5
- no-connect marks 4 -> 0
Changed lines of the file:
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@@
 		(color 0 0 0 0)
 	)
-	(no_connect
-		(at 121.92 63.5)
-	)
-	(no_connect
-		(at 121.92 73.66)
-	)
-	(no_connect
-		(at 121.92 66.04)
-	)
-	(no_connect
-		(at 121.92 60.96)
-	)
 	(wire
 		(pts
@@
 	(wire
 		(pts
-			(xy 121.92 68.58) (xy 101.6 68.58)
-		)
-		(stroke
-			(width 0)
-			(type default)
-		)
-	)
-	(wire
-		(pts
 			(xy 121.92 58.42) (xy 101.6 58.42)
 		)
@@
 		(pts
 			(xy 121.92 66.04) (xy 101.6 66.04)
+		)
+		(stroke
+			(width 0)
+			(type default)
+		)
+	)
+	(wire
+		(pts
+			(xy 101.6 68.58) (xy 121.92 68.58)
 		)
 		(stroke
@@
 		)
 	)
-	(hierarchical_label "MEM_EXP1_CS"
+	(hierarchical_label "EXP_MEM_CS5"
 		(shape output)
 		(at 121.92 71.12 0)
@@
 		)
 	)
+	(hierarchical_label "RAM_BANK2_CS"
+		(shape output)
+		(at 121.92 63.5 0)
+		(effects
+			(font
+				(size 1.27 1.27)
+			)
+			(justify left)
+		)
+	)
 	(hierarchical_label "ROM_CS"
 		(shape output)
@@
 		)
 	)
+	(hierarchical_label "EXP_MEM_CS6"
+		(shape output)
+		(at 121.92 73.66 0)
+		(effects
+			(font
+				(size 1.27 1.27)
+			)
+			(justify left)
+		)
+	)
 	(hierarchical_label "RAM_BANK0_CS"
 		(shape output)
@@
 		)
 	)
-	(hierarchical_label "MEM_EXP0_CS"
+	(hierarchical_label "RAM_BANK4_CS"
 		(shape output)
 		(at 121.92 68.58 0)
+		(effects
+			(font
+				(size 1.27 1.27)
+			)
+			(justify left)
+		)
+	)
+	(hierarchical_label "RAM_BANK3_CS"
+		(shape output)
+		(at 121.92 66.04 0)
 		(effects
 			(font
@@
 			)
 			(justify right)
+		)
+	)
+	(hierarchical_label "RAM_BANK1_CS"
+		(shape output)
+		(at 121.92 60.96 0)
+		(effects
+			(font
+				(size 1.27 1.27)
+			)
+			(justify left)
 		)
 	)
@@
 		(in_pos_files yes)
 		(dnp no)
-		(property "Reference" "C9"
+		(property "Reference" "C7"
 			(at 81.28 40.894 0)
 			(show_name no)
@@
 			)
 		)
-		(property "Footprint" "Capacitor_THT:C_Disc_D5.0mm_W2.5mm_P5.00mm"
+		(property "Footprint" "Capacitor_SMD:C_0805_2012Metric"
 			(at 77.47 47.9552 0)
 			(hide yes)
@@
 			(project "8088-mainboard"
 				(path "/15ce4f45-6f32-456e-874c-aac11293789a/8603fecf-1343-4cbc-8a43-8cc8a41e8f5f"
-					(reference "C9")
+					(reference "C7")
 					(unit 1)
 				)
@@
 		(dnp no)
 		(fields_autoplaced yes)
-		(property "Reference" "#PWR034"
+		(property "Reference" "#PWR035"
 			(at 69.85 73.66 0)
 			(hide yes)
@@
 			(project "8088-mainboard"
 				(path "/15ce4f45-6f32-456e-874c-aac11293789a/8603fecf-1343-4cbc-8a43-8cc8a41e8f5f"
-					(reference "#PWR034")
+					(reference "#PWR035")
 					(unit 1)
 				)
@@
 		(in_pos_files yes)
 		(dnp no)
-		(property "Reference" "#PWR033"
+		(property "Reference" "#PWR034"
 			(at 63.5 74.93 0)
 			(hide yes)
@@
 			(project "8088-mainboard"
 				(path "/15ce4f45-6f32-456e-874c-aac11293789a/8603fecf-1343-4cbc-8a43-8cc8a41e8f5f"
-					(reference "#PWR033")
+					(reference "#PWR034")
 					(unit 1)
 				)
@@
 		(in_pos_files yes)
 		(dnp no)
-		(property "Reference" "#PWR036"
+		(property "Reference" "#PWR037"
 			(at 88.9 45.72 0)
 			(hide yes)
@@
 			(project "8088-mainboard"
 				(path "/15ce4f45-6f32-456e-874c-aac11293789a/8603fecf-1343-4cbc-8a43-8cc8a41e8f5f"
-					(reference "#PWR036")
+					(reference "#PWR037")
 					(unit 1)
 				)
@@
 		(dnp no)
 		(fields_autoplaced yes)
-		(property "Reference" "#PWR035"
+		(property "Reference" "#PWR036"
 			(at 71.12 46.99 0)
 			(hide yes)
@@
 			(project "8088-mainboard"
 				(path "/15ce4f45-6f32-456e-874c-aac11293789a/8603fecf-1343-4cbc-8a43-8cc8a41e8f5f"
-					(reference "#PWR035")
+					(reference "#PWR036")
 					(unit 1)
 				)
@@
 		(dnp no)
 		(fields_autoplaced yes)
-		(property "Reference" "#PWR037"
+		(property "Reference" "#PWR038"
 			(at 88.9 90.17 0)
 			(hide yes)
@@
 			(project "8088-mainboard"
 				(path "/15ce4f45-6f32-456e-874c-aac11293789a/8603fecf-1343-4cbc-8a43-8cc8a41e8f5f"
-					(reference "#PWR037")
+					(reference "#PWR038")
 					(unit 1)
 				)

Commit message: Update schema
Other:
- moved on the sheet: C7, U6
