File: hardware/kicad/MEM_DECODER.kicad_sch (KiCad schematic)
At the start: 2 parts, among them U6 74LS138

Commit message: Add mainboard v2.0 (#6)
* Add mainboard v2.0
Parts:
- C7: renamed from C9; footprint Capacitor_THT:C_Disc_D5.0mm_W2.5mm_P5.00mm -> Capacitor_SMD:C_0805_2012Metric
Connections:
- net RAM_BANK3_CS: now reaches U6.12 (O3)
- net RAM_BANK2_CS: now reaches U6.13 (O2)
- net RAM_BANK1_CS: now reaches U6.14 (O1)
- net EXP_MEM_CS6: now reaches U6.9 (O6)
- net MEM_EXP0_CS renamed RAM_BANK4_CS
- net MEM_EXP1_CS renamed EXP_MEM_CS5
- no-connect marks 4 -> 0
Other:
- moved on the sheet: C7, U6
