File: hardware/kicad/PIC.kicad_sch (KiCad schematic)
At the start: 11 parts, among them J10 Conn_01x04, U15 8259A-2

Commit message: Update schema
Other:
- moved on the sheet: J10
Changed lines of the file:
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@@
 	(hierarchical_label "IO_PIC_CS"
 		(shape input)
-		(at 66.04 152.4 180)
+		(at 39.37 170.18 180)
 		(effects
 			(font
@@
 	(hierarchical_label "INTR"
 		(shape output)
-		(at 66.04 154.94 180)
+		(at 39.37 172.72 180)
 		(effects
 			(font
@@
 	(hierarchical_label "INTA"
 		(shape input)
-		(at 66.04 157.48 180)
+		(at 39.37 175.26 180)
 		(effects
 			(font
@@
 	(symbol
 		(lib_id "Connector_Generic:Conn_01x04")
-		(at 71.12 152.4 0)
+		(at 44.45 170.18 0)
 		(unit 1)
 		(body_style 1)
@@
 		(fields_autoplaced yes)
 		(property "Reference" "J10"
-			(at 73.66 152.3999 0)
+			(at 46.99 170.1799 0)
 			(show_name no)
 			(do_not_autoplace no)
@@
 		)
 		(property "Value" "Conn_01x04"
-			(at 73.66 154.9399 0)
+			(at 46.99 172.7199 0)
 			(show_name no)
 			(do_not_autoplace no)
@@
 		)
 		(property "Footprint" "Connector_PinHeader_2.54mm:PinHeader_1x04_P2.54mm_Vertical"
-			(at 71.12 152.4 0)
-			(hide yes)
-			(show_name no)
-			(do_not_autoplace no)
-			(effects
-				(font
-					(size 1.27 1.27)
-				)
-			)
-		)
-		(property "Datasheet" ""
-			(at 71.12 152.4 0)
+			(at 44.45 170.18 0)
+			(hide yes)
+			(show_name no)
+			(do_not_autoplace no)
+			(effects
+				(font
+					(size 1.27 1.27)
+				)
+			)
+		)
+		(property "Datasheet" ""
+			(at 44.45 170.18 0)
 			(hide yes)
 			(show_name no)
@@
 		)
 		(property "Description" "Generic connector, single row, 01x04, script generated (kicad-library-utils/schlib/autogen/connector/)"
-			(at 71.12 152.4 0)
+			(at 44.45 170.18 0)
 			(hide yes)
 			(show_name no)
@@
 	(symbol
 		(lib_id "power:GND")
-		(at 66.04 149.86 270)
+		(at 39.37 167.64 270)
 		(mirror x)
 		(unit 1)
@@
 		(dnp no)
 		(property "Reference" "#PWR0113"
-			(at 59.69 149.86 0)
+			(at 33.02 167.64 0)
 			(hide yes)
 			(show_name no)
@@
 		)
 		(property "Value" "GND"
-			(at 61.976 149.86 0)
+			(at 35.306 167.64 0)
 			(show_name no)
 			(do_not_autoplace no)
@@
 		)
 		(property "Footprint" ""
-			(at 66.04 149.86 0)
-			(hide yes)
-			(show_name no)
-			(do_not_autoplace no)
-			(effects
-				(font
-					(size 1.27 1.27)
-				)
-			)
-		)
-		(property "Datasheet" ""
-			(at 66.04 149.86 0)
+			(at 39.37 167.64 0)
+			(hide yes)
+			(show_name no)
+			(do_not_autoplace no)
+			(effects
+				(font
+					(size 1.27 1.27)
+				)
+			)
+		)
+		(property "Datasheet" ""
+			(at 39.37 167.64 0)
 			(hide yes)
 			(show_name no)
@@
 		)
 		(property "Description" "Power symbol creates a global label with name \"GND\" , ground"
-			(at 66.04 149.86 0)
-			(hide yes)
-			(show_name no)
+			(at 39.37 167.64 0)
+			(hide yes)
+			(show_name no)
