File: hardware/kicad/PIT.kicad_sch (KiCad schematic)
At the start: 14 parts, among them J2 Ext Res, J3 Ext CLK, SW2 Reset, U5 8284, Y1 14.31818 MHz

Commit message: Add mainboard v2.0
Parts:
- removed C5: 10 uF, Capacitor_THT:CP_Radial_D4.0mm_P1.50mm, symbol Device:C
- removed C6: 100 nF, Capacitor_SMD:C_0805_2012Metric, symbol Device:C
- removed D1: RST LED, LED_SMD:LED_0805_2012Metric, symbol Device:LED
- removed J2: Ext Res, Connector_PinHeader_2.54mm:PinHeader_1x02_P2.54mm_Vertical, symbol Connector_Generic:Conn_01x02
- removed J3: Ext CLK, Connector_PinHeader_2.54mm:PinHeader_1x02_P2.54mm_Vertical, symbol Connector_Generic:Conn_01x02
- removed R4: 680, Resistor_SMD:R_0805_2012Metric, symbol Device:R
- removed R5, R6, R7, R9: 10k, Resistor_SMD:R_0805_2012Metric, symbol Device:R
- removed R8: 1k, Resistor_SMD:R_0805_2012Metric, symbol Device:R
- removed SW2: Reset, Button_Switch_THT:SW_PUSH_6mm, symbol Switch:SW_Push
- removed U5: 8284, Package_DIP:DIP-18_W7.62mm_Socket, symbol Timer:8284
- removed Y1: 14.31818 MHz, Crystal:Crystal_HC49-U_Vertical, symbol Device:Crystal
- added C20, C21: 100nF, Capacitor_SMD:C_0805_2012Metric, symbol Device:C
- added J11: Conn_01x04, Connector_PinHeader_2.54mm:PinHeader_1x04_P2.54mm_Vertical, symbol Connector_Generic:Conn_01x04
- added U16: 8254, Package_DIP:DIP-24_W15.24mm_Socket, symbol Timer:8254
- added U17: 74LS74, Package_DIP:DIP-14_W7.62mm_Socket, symbol 74xx:74LS74
Connections:
- net GND: now also C20.2, C21.2, J11.1 (Pin_1), U16.12 (GND), U16.14 (G1), U16.15 (CLK1), U16.16 (G2), U16.18 (CLK2), U17.11 (C), U17.12 (D), U17.7 (GND)
- net PCLK: now also U17.3 (C)
- net VCC: now also C20.1, C21.1, U16.11 (G0), U16.24 (VCC), U17.1 (~{R}), U17.10 (~{S}), U17.13 (~{R}), U17.14 (VCC), U17.4 (~{S})
- new net: U17.2 (D), U17.6 (~{Q})
- new net A0: U16.19 (A0)
- new net A1: U16.20 (A1)
- new net CLK0: J11.3 (Pin_3), U16.9 (CLK0), U17.5 (Q)
- new net D0: U16.8 (D0)
- new net D1: U16.7 (D1)
- new net D2: U16.6 (D2)
- new net D3: U16.5 (D3)
- new net D4: U16.4 (D4)
- new net D5: U16.3 (D5)
- new net D6: U16.2 (D6)
- new net D7: U16.1 (D7)
- new net IO_PIT_CS: J11.2 (Pin_2), U16.21 (~{CS})
- new net PIT_IRQ: J11.4 (Pin_4), U16.10 (OUT0)
- new net RD: U16.22 (~{RD})
- new net WR: U16.23 (~{WR})
- no-connect marks 1 -> 4

Commit message: Update schema
Other:
- moved on the sheet: C20, C21, J11, U16, U17A, U17B, U17C
