File: hardware/kicad/POWER.kicad_sch (KiCad schematic)
At the start: 10 parts, among them J4 POWER 5v, Q1 NDP6020P

Commit message: Add mainboard v2.0
Parts:
- D2: renamed from D1; footprint LED_THT:LED_D3.0mm -> LED_SMD:LED_0805_2012Metric
- R11: renamed from R4; footprint Resistor_THT:R_Axial_DIN0207_L6.3mm_D2.5mm_P7.62mm_Horizontal -> Resistor_SMD:R_0805_2012Metric
- R12: renamed from R5; footprint Resistor_THT:R_Axial_DIN0207_L6.3mm_D2.5mm_P7.62mm_Horizontal -> Resistor_SMD:R_0805_2012Metric
- renumbered C13 to C15, J4 to J8
Changed lines of the file:
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@@
 		(dnp no)
 		(fields_autoplaced yes)
-		(property "Reference" "#PWR056"
+		(property "Reference" "#PWR086"
 			(at 46.99 82.55 0)
 			(hide yes)
@@
 			(project "8088-mainboard"
 				(path "/15ce4f45-6f32-456e-874c-aac11293789a/e9d836d6-3c3a-4b6e-a562-389c64894272"
-					(reference "#PWR056")
+					(reference "#PWR086")
 					(unit 1)
 				)
@@
 		(in_pos_files yes)
 		(dnp no)
-		(property "Reference" "#PWR065"
+		(property "Reference" "#PWR095"
 			(at 147.32 133.35 0)
 			(hide yes)
@@
 			(project "8088-mainboard"
 				(path "/15ce4f45-6f32-456e-874c-aac11293789a/e9d836d6-3c3a-4b6e-a562-389c64894272"
-					(reference "#PWR065")
+					(reference "#PWR095")
 					(unit 1)
 				)
@@
 		(in_pos_files yes)
 		(dnp no)
-		(property "Reference" "#PWR062"
+		(property "Reference" "#PWR092"
 			(at 128.27 83.82 0)
 			(hide yes)
@@
 			(project "8088-mainboard"
 				(path "/15ce4f45-6f32-456e-874c-aac11293789a/e9d836d6-3c3a-4b6e-a562-389c64894272"
-					(reference "#PWR062")
+					(reference "#PWR092")
 					(unit 1)
 				)
@@
 		(in_pos_files yes)
 		(dnp no)
-		(property "Reference" "#PWR059"
+		(property "Reference" "#PWR089"
 			(at 74.93 120.65 0)
 			(hide yes)
@@
 			(project "8088-mainboard"
 				(path "/15ce4f45-6f32-456e-874c-aac11293789a/e9d836d6-3c3a-4b6e-a562-389c64894272"
-					(reference "#PWR059")
+					(reference "#PWR089")
 					(unit 1)
 				)
@@
 		(in_pos_files yes)
 		(dnp no)
-		(property "Reference" "#PWR060"
+		(property "Reference" "#PWR090"
 			(at 78.74 97.79 0)
 			(hide yes)
@@
 			(project "8088-mainboard"
 				(path "/15ce4f45-6f32-456e-874c-aac11293789a/e9d836d6-3c3a-4b6e-a562-389c64894272"
-					(reference "#PWR060")
+					(reference "#PWR090")
 					(unit 1)
 				)
@@
 		(in_pos_files yes)
 		(dnp no)
-		(property "Reference" "#PWR064"
+		(property "Reference" "#PWR094"
 			(at 147.32 120.65 0)
 			(hide yes)
@@
 			(project "8088-mainboard"
 				(path "/15ce4f45-6f32-456e-874c-aac11293789a/e9d836d6-3c3a-4b6e-a562-389c64894272"
-					(reference "#PWR064")
+					(reference "#PWR094")
 					(unit 1)
 				)
@@
 		(in_pos_files yes)
 		(dnp no)
-		(property "Reference" "#PWR063"
+		(property "Reference" "#PWR093"
 			(at 140.97 93.98 0)
 			(hide yes)
@@
 			(project "8088-mainboard"
 				(path "/15ce4f45-6f32-456e-874c-aac11293789a/e9d836d6-3c3a-4b6e-a562-389c64894272"
-					(reference "#PWR063")
+					(reference "#PWR093")
 					(unit 1)
 				)
@@
 		(in_pos_files yes)
 		(dnp no)
-		(property "Reference" "#PWR066"
+		(property "Reference" "#PWR096"
 			(at 177.8 120.65 0)
 			(hide yes)
@@
 			(project "8088-mainboard"
 				(path "/15ce4f45-6f32-456e-874c-aac11293789a/e9d836d6-3c3a-4b6e-a562-389c64894272"
-					(reference "#PWR066")
+					(reference "#PWR096")
 					(unit 1)
 				)
@@
 		(in_pos_files yes)
 		(dnp no)
-		(property "Reference" "#PWR058"
+		(property "Reference" "#PWR088"
 			(at 74.93 97.79 0)
 			(hide yes)
@@
 			(project "8088-mainboard"
 				(path "/15ce4f45-6f32-456e-874c-aac11293789a/e9d836d6-3c3a-4b6e-a562-389c64894272"
-					(reference "#PWR058")
+					(reference "#PWR088")
 					(unit 1)
 				)
@@
 		(in_pos_files yes)
 		(dnp no)
-		(property "Reference" "C13"
+		(property "Reference" "C15"
 			(at 68.072 110.49 90)
 			(show_name no)
@@
 			(project "8088-mainboard"
 				(path "/15ce4f45-6f32-456e-874c-aac11293789a/e9d836d6-3c3a-4b6e-a562-389c64894272"
-					(reference "C13")
+					(reference "C15")
 					(unit 1)
 				)
@@
 		(in_pos_files yes)
 		(dnp no)
-		(property "Reference" "#PWR067"
+		(property "Reference" "#PWR097"
 			(at 177.8 133.35 0)
 			(hide yes)
@@
 			(project "8088-mainboard"
 				(path "/15ce4f45-6f32-456e-874c-aac11293789a/e9d836d6-3c3a-4b6e-a562-389c64894272"
-					(reference "#PWR067")
+					(reference "#PWR097")
 					(unit 1)
 				)
@@
 		(dnp no)
 		(fields_autoplaced yes)
-		(property "Reference" "#PWR057"
+		(property "Reference" "#PWR087"
 			(at 46.99 100.33 0)
 			(hide yes)
@@
 			(project "8088-mainboard"
 				(path "/15ce4f45-6f32-456e-874c-aac11293789a/e9d836d6-3c3a-4b6e-a562-389c64894272"
-					(reference "#PWR057")
+					(reference "#PWR087")
 					(unit 1)
 				)
@@
 		(dnp no)
 		(fields_autoplaced yes)
-		(property "Reference" "J4"
+		(property "Reference" "J8"
 			(at 105.41 82.5499 90)
 			(show_name no)
@@
 			(project "8088-mainboard"
 				(path "/15ce4f45-6f32-456e-874c-aac11293789a/e9d836d6-3c3a-4b6e-a562-389c64894272"
-					(reference "J4")
+					(reference "J8")
 					(unit 1)
 				)
@@
 		(dnp no)
 		(fields_autoplaced yes)
-		(property "Reference" "D1"
+		(property "Reference" "D2"
 			(at 50.8 90.4874 90)
 			(show_name no)
@@
 			)
 		)
-		(property "Footprint" "LED_THT:LED_D3.0mm"
+		(property "Footprint" "LED_SMD:LED_0805_2012Metric"
 			(at 46.99 90.17 0)
 			(hide yes)
@@
 			(project "8088-mainboard"
 				(path "/15ce4f45-6f32-456e-874c-aac11293789a/e9d836d6-3c3a-4b6e-a562-389c64894272"
-					(reference "D1")
+					(reference "D2")
 					(unit 1)
 				)
@@
 		(in_pos_files yes)
 		(dnp no)
-		(property "Reference" "R5"
+		(property "Reference" "R12"
 			(at 88.9 93.726 0)
 			(show_name no)
@@
 			)
 		)
-		(property "Footprint" "Resistor_THT:R_Axial_DIN0207_L6.3mm_D2.5mm_P7.62mm_Horizontal"
+		(property "Footprint" "Resistor_SMD:R_0805_2012Metric"
 			(at 88.9 96.012 90)
 			(hide yes)
@@
 			(project "8088-mainboard"
 				(path "/15ce4f45-6f32-456e-874c-aac11293789a/e9d836d6-3c3a-4b6e-a562-389c64894272"
-					(reference "R5")
+					(reference "R12")
 					(unit 1)
 				)
@@
 		(in_pos_files yes)
 		(dnp no)
-		(property "Reference" "#PWR061"
+		(property "Reference" "#PWR091"
 			(at 114.3 106.68 0)
 			(hide yes)
@@
 			(project "8088-mainboard"
 				(path "/15ce4f45-6f32-456e-874c-aac11293789a/e9d836d6-3c3a-4b6e-a562-389c64894272"
-					(reference "#PWR061")
+					(reference "#PWR091")
 					(unit 1)
 				)
@@
 		(in_pos_files yes)
 		(dnp no)
-		(property "Reference" "R4"
+		(property "Reference" "R11"
 			(at 42.926 82.55 0)
 			(show_name no)
@@
 			)
 		)
-		(property "Footprint" "Resistor_THT:R_Axial_DIN0207_L6.3mm_D2.5mm_P7.62mm_Horizontal"
+		(property "Footprint" "Resistor_SMD:R_0805_2012Metric"
 			(at 45.212 82.55 90)
 			(hide yes)
@@
 			(project "8088-mainboard"
 				(path "/15ce4f45-6f32-456e-874c-aac11293789a/e9d836d6-3c3a-4b6e-a562-389c64894272"
-					(reference "R4")
-					(unit 1)
-				)
+					(reference "R11")
+					(unit 1)
+				)

Commit message: Update schema
Other:
- moved on the sheet: C15, D2, H1, H2, H3, H4, J8, Q1, R11, R12
