File: hardware/kicad/POWER.kicad_sch (KiCad schematic)
At the start: 10 parts, among them J4 POWER 5v, Q1 NDP6020P

Commit message: Add mainboard v2.0 (#6)
* Add mainboard v2.0
Parts:
- D2: renamed from D1; footprint LED_THT:LED_D3.0mm -> LED_SMD:LED_0805_2012Metric
- R11: renamed from R4; footprint Resistor_THT:R_Axial_DIN0207_L6.3mm_D2.5mm_P7.62mm_Horizontal -> Resistor_SMD:R_0805_2012Metric
- R12: renamed from R5; footprint Resistor_THT:R_Axial_DIN0207_L6.3mm_D2.5mm_P7.62mm_Horizontal -> Resistor_SMD:R_0805_2012Metric
- renumbered C13 to C15, J4 to J8
Other:
- moved on the sheet: C15, D2, H1, H2, H3, H4, J8, Q1, R11, R12
