File: hardware/kicad/display-module/display-module.kicad_sch (KiCad schematic)
At the start: 8 parts, among them J1 Exp0, U1 74LS00, U2 74LS373

Commit message: Add mainboard v2.0
Parts:
- removed J1: Exp0, Connector_PinSocket_2.54mm:PinSocket_2x20_P2.54mm_Vertical, symbol Connector_Generic:Conn_02x20_Odd_Even
- added C1: 220 uF, Capacitor_THT:CP_Radial_D5.0mm_P2.00mm, symbol Device:C
- added J1: EXP_0_A, Connector_PinHeader_2.54mm:PinHeader_2x20_P2.54mm_Horizontal, symbol Connector_Generic:Conn_02x20_Counter_Clockwise
- added J2: EXP_0_B, Connector_PinHeader_2.54mm:PinHeader_2x10_P2.54mm_Horizontal, symbol Connector_Generic:Conn_02x10_Counter_Clockwise
- DS1: value WC1602A -> WC1604A; footprint Connector_PinSocket_2.54mm:PinSocket_1x16_P2.54mm_Vertical -> Connector_PinHeader_2.54mm:PinHeader_1x16_P2.54mm_Horizontal
- renumbered R2 to R1, U2 to U1, U1 to U2
Connections:
- net A0: now also J1.40 (Pin_40)
- net A1: now also J1.39 (Pin_39)
- net A10: now also J1.30 (Pin_30)
- net A11: now also J1.29 (Pin_29)
- net A12: now also J1.28 (Pin_28)
- net A13: now also J1.27 (Pin_27)
- net A14: now also J1.26 (Pin_26)
- net A15: now also J1.25 (Pin_25)
- net A16: now also J1.24 (Pin_24)
- net A17: now also J1.23 (Pin_23)
- net A18: now also J1.22 (Pin_22)
- net A19: now also J1.21 (Pin_21)
- net A2: now also J1.38 (Pin_38)
- net A3: now also J1.37 (Pin_37)
- net A4: now also J1.36 (Pin_36)
- net A5: now also J1.35 (Pin_35)
- net A6: now also J1.34 (Pin_34)
- net A7: now also J1.33 (Pin_33)
- net A8: now also J1.32 (Pin_32)
- net A9: now also J1.31 (Pin_31)
- net ALE: now also J1.9 (Pin_9)
- net CLK: now also J2.2 (Pin_2)
- net D0: now also J1.18 (Pin_18)
- net D1: now also J1.17 (Pin_17)
- net D2: now also J1.16 (Pin_16)
- net D3: now also J1.15 (Pin_15)
- net D4: now also J1.14 (Pin_14)
- net D5: now also J1.13 (Pin_13)
- net D6: now also J1.12 (Pin_12)
- net D7: now also J1.11 (Pin_11)
- net GND: now also C1.2, J1.1 (Pin_1), J1.10 (Pin_10), J1.19 (Pin_19), J1.20 (Pin_20), J2.1 (Pin_1), J2.10 (Pin_10), J2.19 (Pin_19), J2.20 (Pin_20)
- net IOM: now also J1.3 (Pin_3)
- net RD: now also J1.5 (Pin_5)
- net RDY: now also J1.6 (Pin_6)
- net RESET: now also J1.7 (Pin_7)
- net VCC: now also C1.1, J1.2 (Pin_2)
- net WR: now also J1.4 (Pin_4)
- net IO_EXP_CS renamed EXP_IO_CS4
- net EXP_IO_CS4: now also J2.7 (Pin_7)
- new net DEN: J2.6 (Pin_6)
- new net DT_R: J2.5 (Pin_5)
- new net EXP_IO_CS5: J2.8 (Pin_8)
- new net EXP_IO_CS6: J2.9 (Pin_9)
- new net EXP_IRQ1: J2.13 (Pin_13)
- new net EXP_IRQ2: J2.14 (Pin_14)
- new net EXP_IRQ3: J2.15 (Pin_15)
- new net EXP_IRQ5: J2.16 (Pin_16)
- new net EXP_IRQ6: J2.17 (Pin_17)
- new net EXP_IRQ7: J2.18 (Pin_18)
- new net EXP_MEM_CS5: J2.11 (Pin_11)
- new net EXP_MEM_CS6: J2.12 (Pin_12)
- new net HLDA: J2.4 (Pin_4)
- new net HOLD: J2.3 (Pin_3)
- new net NMI: J1.8 (Pin_8)
Other:
- moved on the sheet: C2, DS1, R1, RV1, U1, U2A, U2B, U2C, U2D

Commit message: Update mainboard and expansion modules
Parts:
- removed U2: 74LS00, Package_DIP:DIP-14_W7.62mm_Socket, symbol 74xx:74LS00
- added H1: MountingHole_Pad, MountingHole:MountingHole_3.2mm_M3_Pad, symbol Mechanical:MountingHole_Pad
- added JP1, JP2: Jumper_2_Small_Open, Jumper:SolderJumper-2_P1.3mm_Open_Pad1.0x1.5mm, symbol Jumper:Jumper_2_Small_Open
- added U2: 74LS02, Package_DIP:DIP-14_W7.62mm_Socket, symbol 74xx:74LS02
Connections:
- net EXP_IO_CS4: now also JP1.1 (A)
- net EXP_IO_CS5: now also JP2.1 (A)
- net GND: now also H1.1, U2.11, U2.12, U2.5, U2.6, U2.7 (GND), U2.8, U2.9
- net LCD_WRITE: now also U2.1
- net VCC: now also U2.14 (VCC)
- net WR: now also U2.3
- new net DISPLAY_IO_CS: JP1.2 (B), JP2.2 (B), U2.2
- no-connect marks 0 -> 3
Other:
- moved on the sheet: C2, DS1, R1, RV1, U1
