File: hardware/kicad/smart-io-module/smart-io-module.kicad_pcb (KiCad board)
At the start: 2 copper layers, 121.9 x 73.7 mm, 45 parts, among them J1 TFT, J2 SD, J3 EXP_A, J4 EXP_B, U1 ESP32-S3-DevKitC, U2 74HC595, U3 74LS02, U4 74LS373, U5 SN74LVC245AN, U6 SN74LVC245AN, U7 SN74LVC245AN, U8 74LS373

Commit message: Update mainboard and expansion modules
Parts:
- C3, C5: moved to F.Cu
- moved R2 45.4 mm to (117.8, 53.3), turned to 180 degrees
- moved R3 41.8 mm to (117.8, 58.4), turned to 180 degrees
- moved R4 40.9 mm to (117.8, 55.9), turned to 180 degrees
- moved C2 39.9 mm to (109.5, 83.8)
- moved C6 39.9 mm to (109.5, 99.1)
- moved U4 38.7 mm to (114.3, 91.4)
- moved U5 38.7 mm to (149.9, 106.7)
- moved U7 38.7 mm to (149.9, 91.4)
- moved U8 38.7 mm to (114.3, 106.7)
- moved R1 37.6 mm to (117.8, 61.0), turned to 0 degrees
- moved C3 37.5 mm to (145.1, 99.1)
- moved C5 37.5 mm to (145.1, 83.8)
- moved R9 13.0 mm to (188.0, 108.3)
- moved D1 8.89 mm to (200.1, 62.2)
- moved R11 8.03 mm to (185.4, 108.3)
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Connections:
- U1 pad 10: /ESP_D_OUT6 -> /ESP_D_IN6
- U1 pad 11: /ESP_HLDA -> /ESP_D_IN7
- U1 pad 12: /ESP_D_IN7 -> /ESP_CTRL_SER
- U1 pad 27: /ESP_IO_CS -> /ESP_HLDA
- U1 pad 29: /ESP_D_IN0 -> /ESP_D_OUT7
- U1 pad 30: /ESP_D_OUT7 -> /ESP_D_OUT6
- U1 pad 31: /ESP_CTRL_SER -> /ESP_CTRL_EN
- U1 pad 35: /ESP_D_IN6 -> /ESP_IO_CS
- U1 pad 36: /ESP_D_IN5 -> /ESP_D_OUT5
- U1 pad 37: /ESP_D_IN4 -> /ESP_D_OUT4
- U1 pad 38: /ESP_D_IN3 -> /ESP_D_OUT3
- U1 pad 39: /ESP_D_IN2 -> /ESP_D_OUT2
- U1 pad 4: /ESP_D_OUT0 -> /ESP_D_IN0
- U1 pad 40: /ESP_D_IN1 -> /ESP_D_OUT1
- U1 pad 41: /ESP_CTRL_EN -> /ESP_D_OUT0
- U1 pad 5: /ESP_D_OUT1 -> /ESP_D_IN1
- U1 pad 6: /ESP_D_OUT2 -> /ESP_D_IN2
- U1 pad 7: /ESP_D_OUT3 -> /ESP_D_IN3
- U1 pad 8: /ESP_D_OUT4 -> /ESP_D_IN4
- U1 pad 9: /ESP_D_OUT5 -> /ESP_D_IN5
Routing:
- net /ESP_D_OUT1: track 0.00 -> 108.6 mm
- net /ESP_D_OUT2: track 0.00 -> 107.7 mm
- net Net-(D4-K): track 0.00 -> 103.9 mm, vias 0 -> 1
- net /ESP_D_OUT0: track 0.00 -> 103.7 mm
- net Net-(U4-LE): track 0.00 -> 84.0 mm, vias 0 -> 2
- net VCC: track 152.8 -> 229.9 mm, vias 3 -> 1
- net /ESP_CTRL_EN: track 0.00 -> 76.2 mm, vias 0 -> 1
- net /ESP_D_OUT6: track 0.00 -> 70.4 mm, vias 0 -> 1
- net /ESP_D_OUT7: track 0.00 -> 70.4 mm, vias 0 -> 1
- net /ESP_CTRL_SER: track 0.00 -> 64.2 mm
- net /ESP_CTRL_RCLK: track 0.00 -> 63.9 mm, vias 0 -> 1
- net /D0: track 38.0 -> 100.0 mm, vias 0 -> 2
- net /ESP_DATA_LATCH: track 13.3 -> 72.5 mm, vias 0 -> 1
- net Net-(U5-B8): track 0.00 -> 57.8 mm
- net /ESP_D_OUT5: track 0.00 -> 56.9 mm
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
Commit message: Update mainboard and expansion modules
Parts:
- U1: value ESP32-S3-DevKitC -> ESP32-S3; footprint PCM_Espressif:ESP32-S3-DevKitC -> Module:ESP32-S3-Dual-Type-C
- moved R8 7.62 mm to (188.0, 65.1)
- moved U1 7.10 mm to (154.3, 72.4)
- moved D1 6.50 mm to (205.7, 65.5), turned to 90 degrees
- moved C1 1.27 mm to (109.5, 66.0)
Routing:
- net /ESP_HLDA: track 55.9 -> 39.8 mm, vias 2 -> 0
- net /ESP_CTRL_SRCLK: track 34.1 -> 49.0 mm, vias 1 -> 0
- net /ESP_IO_CS: track 76.2 -> 61.5 mm
- net /ESP_CTRL_EN: track 76.2 -> 88.9 mm
- net /3V3: track 205.4 -> 217.1 mm
- net /ESP_CTRL_SER: track 64.2 -> 75.8 mm
- net /ESP_D_OUT1: track 108.6 -> 119.6 mm
- net /ESP_D_OUT0: track 103.7 -> 114.6 mm
- net /ESP_CTRL_RCLK: track 63.9 -> 74.6 mm
- net /ESP_D_OUT2: track 107.7 -> 117.3 mm
- net /ESP_DATA_LATCH: track 72.5 -> 80.5 mm
- net Net-(D3-K): track 51.9 -> 45.1 mm
- net /ESP_D_OUT4: track 56.9 -> 62.6 mm
- net /ESP_D_OUT5: track 56.9 -> 62.6 mm
- net /ESP_D_OUT3: track 56.9 -> 62.6 mm
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