File: hardware/kicad/smart-io-module/smart-io-module.kicad_sch (KiCad schematic)
At the start: 27 parts, among them J1 TFT, J2 SD, U1 ESP32-S3-DevKitC, U2 74HC595, U3 74LS02, U4 74LS373, U5 SN74LVC245AN, U6 SN74LVC245AN, U7 SN74LVC245AN, U8 74LS373

Commit message: Update mainboard and expansion modules
Connections:
- net ESP_CTRL_EN: now also U1.31 (GPIO0); no longer U1.41 (GPIO1/ADC1_CH0)
- net ESP_CTRL_SER: now also U1.12 (GPIO8/ADC1_CH7); no longer U1.31 (GPIO0)
- net ESP_D_IN0: now also U1.4 (GPIO4/ADC1_CH3); no longer U1.29 (GPIO48)
- net ESP_D_IN1: now also U1.5 (GPIO5/ADC1_CH4); no longer U1.40 (GPIO2/ADC1_CH1)
- net ESP_D_IN2: now also U1.6 (GPIO6/ADC1_CH5); no longer U1.39 (GPIO42/MTMS)
- net ESP_D_IN3: now also U1.7 (GPIO7/ADC1_CH6); no longer U1.38 (GPIO41/MTDI)
- net ESP_D_IN4: now also U1.8 (GPIO15/ADC2_CH4/32K_P); no longer U1.37 (GPIO40/MTDO)
- net ESP_D_IN5: now also U1.9 (GPIO16/ADC2_CH5/32K_N); no longer U1.36 (GPIO39/MTCK)
- net ESP_D_IN6: now also U1.10 (GPIO17/ADC2_CH6); no longer U1.35 (GPIO38)
- net ESP_D_IN7: now also U1.11 (GPIO18/ADC2_CH7); no longer U1.12 (GPIO8/ADC1_CH7)
- net ESP_D_OUT0: now also U1.41 (GPIO1/ADC1_CH0); no longer U1.4 (GPIO4/ADC1_CH3)
- net ESP_D_OUT1: now also U1.40 (GPIO2/ADC1_CH1); no longer U1.5 (GPIO5/ADC1_CH4)
- net ESP_D_OUT2: now also U1.39 (GPIO42/MTMS); no longer U1.6 (GPIO6/ADC1_CH5)
- net ESP_D_OUT3: now also U1.38 (GPIO41/MTDI); no longer U1.7 (GPIO7/ADC1_CH6)
- net ESP_D_OUT4: now also U1.37 (GPIO40/MTDO); no longer U1.8 (GPIO15/ADC2_CH4/32K_P)
- net ESP_D_OUT5: now also U1.36 (GPIO39/MTCK); no longer U1.9 (GPIO16/ADC2_CH5/32K_N)
- net ESP_D_OUT6: now also U1.30 (GPIO45); no longer U1.10 (GPIO17/ADC2_CH6)
- net ESP_D_OUT7: now also U1.29 (GPIO48); no longer U1.30 (GPIO45)
- net ESP_HLDA: now also U1.27 (GPIO21); no longer U1.11 (GPIO18/ADC2_CH7)
- net ESP_IO_CS: now also U1.35 (GPIO38); no longer U1.27 (GPIO21)
Other:
- moved on the sheet: R2, R3, R4

Commit message: Update mainboard and expansion modules
Parts:
- U1: value ESP32-S3-DevKitC -> ESP32-S3; footprint PCM_Espressif:ESP32-S3-DevKitC -> Module:ESP32-S3-Dual-Type-C
Changed lines of the file:
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@@
 		(in_pos_files yes)
 		(dnp no)
-		(fields_autoplaced yes)
 		(property "Reference" "U1"
 			(at 94.8533 132.08 0)
@@
 			)
 		)
-		(property "Value" "ESP32-S3-DevKitC"
+		(property "Value" "ESP32-S3"
 			(at 94.8533 134.62 0)
 			(show_name no)
@@
 			)
 		)
-		(property "Footprint" "PCM_Espressif:ESP32-S3-DevKitC"
+		(property "Footprint" "Module:ESP32-S3-Dual-Type-C"
 			(at 92.71 143.51 0)
 			(hide yes)
@@
 			)
 		)
-		(property "Description" "ESP32-S3-DevKitC"
-			(at 92.71 86.36 0)
-			(hide yes)
+		(property "Description" "ESP32-S3-Dual-Type-C"
+			(at 82.804 88.646 0)
 			(show_name no)
 			(do_not_autoplace no)
